File: KiCad/analogFE.kicad_sch (KiCad schematic)
At the start: 24 parts, among them U6 NE5532, U7 NE5532, U8 NE5532

Commit message: Preparing to auto-route
Connections:
- net +9V: no longer C10.2, C11.1, C11.2, C7.2, C9.1, R1.2, R10.1, R2.1, R3.1, R6.2, R7.1, R8.2
- new net -9V: C11.2, R8.2
- new net GND: C10.2, C11.1, C7.2, C9.1, R1.2, R10.1, R2.1, R3.1, R6.2, R7.1
Changed lines of the file:
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@@
-	)
-	(junction
-		(at 196.85 91.44)
-		(diameter 0)
-		(color 0 0 0 0)
 	)
 	(junction
@@
 	)
 	(junction
-		(at 196.85 78.74)
-		(diameter 0)
-		(color 0 0 0 0)
-	)
-	(junction
 		(at 127 93.98)
 		(diameter 0)
@@
 	)
 	(junction
-		(at 196.85 104.14)
-		(diameter 0)
-		(color 0 0 0 0)
-	)
-	(junction
 		(at 137.16 93.98)
 		(diameter 0)
@@
 	(wire
 		(pts
-			(xy 196.85 78.74) (xy 196.85 91.44)
-		)
-		(stroke
-			(width 0)
-			(type default)
-		)
-	)
-	(wire
-		(pts
 			(xy 203.2 96.52) (xy 203.2 91.44)
 		)
@@
 	(wire
 		(pts
-			(xy 196.85 91.44) (xy 203.2 91.44)
-		)
-		(stroke
-			(width 0)
-			(type default)
-		)
-	)
-	(wire
-		(pts
 			(xy 134.62 57.15) (xy 134.62 59.69)
 		)
@@
 		)
 		(stroke
-			(width 0)
-			(type default)
-		)
-	)
-	(wire
-		(pts
-			(xy 196.85 91.44) (xy 196.85 104.14)
-		)
-		(stroke
