File: KiCad/analogFE.kicad_sch (KiCad schematic)
At the start: 0 parts

Commit message: Filled out FE schematic block
Parts:
- added C10, C11: C_Small, symbol Device:C_Small
- added C6, C7, C8, C9: C, symbol Device:C
- added D1: BAT54ADW, Package_TO_SOT_SMD:SOT-363_SC-70-6, symbol Diode:BAT54ADW
- added R1, R10, R2, R3, R4, R5, R6, R7, R8, R9: R_US, symbol Device:R_US
- added U6, U7, U8: NE5532, symbol Amplifier_Operational:NE5532
Connections:
- new net: D1.6 (A), U8.1, U8.2 (-)
- new net: C9.2, R7.2, R8.1, U8.3 (+)
- new net: D1.1 (K), U7.1, U7.2 (-)
- new net: C8.2, R10.2, R9.1, U7.3 (+)
- new net: C7.1, D1.2 (K), D1.6 (A), R5.2, R6.1
- new net: C6.2, R2.2, U6.3 (+)
- new net: R3.2, R4.1, U6.2 (-)
- new net: R4.2, R5.1, U6.1
- new net +9V: C10.1, C10.2, C11.1, C11.2, C7.2, C8.1, C9.1, R1.2, R10.1, R2.1, R3.1, R6.2, R7.1, R8.2, R9.2
- new net Guitar_In: C6.1, R1.1

Commit message: Changed footprints, added powersystem
Parts:
- added TP1, TP2, TP3, TP4: TestPoint, TestPoint:TestPoint_Loop_D2.50mm_Drill1.85mm, symbol Connector:TestPoint
- C10, C11: value C_Small -> 10pF; footprint (none) -> Capacitor_SMD:CP_Elec_5x4.5
- C6: value C -> 0.1uF; footprint (none) -> Capacitor_SMD:CP_Elec_5x4.5
- C7: value C -> 33nF; footprint (none) -> Capacitor_SMD:CP_Elec_5x4.5
- C8, C9: value C -> 1mF; footprint (none) -> Capacitor_SMD:CP_Elec_10x10.5
- R1: value R_US -> 1M; footprint (none) -> Resistor_SMD:R_1206_3216Metric
- R10, R8: value R_US -> 620k; footprint (none) -> Resistor_SMD:R_1206_3216Metric
- R2: value R_US -> 22k; footprint (none) -> Resistor_SMD:R_1206_3216Metric
- R3: value R_US -> 47k; footprint (none) -> Resistor_SMD:R_1206_3216Metric
- R4, R6, R7, R9: value R_US -> 100k; footprint (none) -> Resistor_SMD:R_1206_3216Metric
- R5: value R_US -> 470; footprint (none) -> Resistor_SMD:R_1206_3216Metric
- U6, U7, U8: footprint (none) -> op_amp:D8-L
Connections:
- net at D1.6 (A), U8.1, U8.2 (-): now also TP3.1
- net at D1.1 (K), U7.1, U7.2 (-): now also TP1.1
- net at C7.1, D1.2 (K), D1.6 (A)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: now also TP2.1
- net at R4.2, R5.1, U6.1: now also TP4.1
Other:
- moved on the sheet: C10, C11, C9

Commit message: Pushing PCB, and controls schem
Parts:
- removed D1: BAT54ADW, Package_TO_SOT_SMD:SOT-363_SC-70-6, symbol Diode:BAT54ADW
- added D2: BAT54S, Package_TO_SOT_SMD:SOT-23, symbol Diode:BAT54S
Connections:
- net at TP3.1, U8.1, U8.2 (-): now also D2.1 (A)
- net at TP1.1, U7.1, U7.2 (-): now also D2.2 (K)
- net at C7.1, R5.2, R6.1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: now also D2.3 (COM)
Other:
- moved on the sheet: TP2

Commit message: Luke's commit
Connections:
- net +9V: no longer C10.2, C11.1, C7.2, C9.1, R1.2, R10.1, R2.1, R3.1, R6.2, R7.1
- new net GND: C10.2, C11.1, C7.2, C9.1, R1.2, R10.1, R2.1, R3.1, R6.2, R7.1
Changed lines of the file:
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@@
-	)
-	(junction
-		(at 196.85 91.44)
-		(diameter 0)
-		(color 0 0 0 0)
 	)
 	(junction
@@
 	(wire
 		(pts
-			(xy 196.85 78.74) (xy 196.85 91.44)
-		)
-		(stroke
-			(width 0)
-			(type default)
-		)
-	)
-	(wire
-		(pts
 			(xy 203.2 96.52) (xy 203.2 91.44)
 		)
@@
 	(wire
 		(pts
-			(xy 196.85 91.44) (xy 196.85 104.14)
-		)
-		(stroke
+			(xy 196.85 78.74) (xy 196.85 104.14)
+		)
+		(stroke

Commit message: Best one yet
Parts:
- C10, C11, C6, C7: footprint Capacitor_SMD:CP_Elec_5x4.5 -> Capacitor_SMD:C_0603_1608Metric
- C8, C9: value 1mF -> 1uF; footprint Capacitor_SMD:CP_Elec_10x10.5 -> Capacitor_SMD:C_0603_1608Metric
Connections:
- net +9V: no longer C11.2, R8.2
- new net -9V: C11.2, R8.2
Changed lines of the file:
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@@
 	(text_box "Voltage rails for the front end\n"
 		(exclude_from_sim no)
-		(at 207.01 72.39 0)
+		(at 187.96 61.595 0)
 		(size 25.4 6.35)
 		(margins 0.9525 0.9525 0.9525 0.9525)
@@
 	)
 	(junction
-		(at 196.85 78.74)
-		(diameter 0)
-		(color 0 0 0 0)
-	)
-	(junction
 		(at 127 93.98)
 		(diameter 0)
@@
 	)
 	(junction
-		(at 196.85 104.14)
-		(diameter 0)
-		(color 0 0 0 0)
-	)
-	(junction
 		(at 137.16 93.98)
 		(diameter 0)
@@
 	(wire
 		(pts
-			(xy 196.85 91.44) (xy 203.2 91.44)
-		)
-		(stroke
-			(width 0)
-			(type default)
-		)
-	)
-	(wire
-		(pts
 			(xy 134.62 57.15) (xy 134.62 59.69)
 		)
@@
 	(wire
 		(pts
-			(xy 196.85 78.74) (xy 196.85 104.14)
-		)
-		(stroke
-			(width 0)
-			(type default)
-		)
-	)
-	(wire
-		(pts
 			(xy 140.97 66.04) (xy 140.97 68.58)
 		)
@@
 			)
 		)
-		(property "Footprint" "Capacitor_SMD:CP_Elec_5x4.5"
+		(property "Footprint" "Capacitor_SMD:C_0603_1608Metric"
 			(at 203.2 99.06 0)
 			(hide yes)
@@
 			)
 		)
-		(property "Footprint" "Capacitor_SMD:CP_Elec_5x4.5"
+		(property "Footprint" "Capacitor_SMD:C_0603_1608Metric"
 			(at 71.12 95.5548 0)
 			(hide yes)
@@
 			)
 		)
-		(property "Value" "1mF"
+		(property "Value" "1uF"
 			(at 144.272 116.078 0)
 			(show_name no)
@@
 			)
 		)
-		(property "Footprint" "Capacitor_SMD:CP_Elec_10x10.5"
+		(property "Footprint" "Capacitor_SMD:C_0603_1608Metric"
 			(at 141.9352 120.65 0)
 			(hide yes)
@@
 			)
 		)
-		(property "Footprint" "Capacitor_SMD:CP_Elec_5x4.5"
+		(property "Footprint" "Capacitor_SMD:C_0603_1608Metric"
 			(at 203.2 83.82 0)
 			(hide yes)
@@
 			)
 		)
-		(property "Footprint" "Capacitor_SMD:CP_Elec_5x4.5"
+		(property "Footprint" "Capacitor_SMD:C_0603_1608Metric"
 			(at 127.9652 101.6 0)
 			(hide yes)
@@
 			)
 		)
-		(property "Value" "1mF"
+		(property "Value" "1uF"
 			(at 144.018 61.214 0)
 			(show_name no)
@@
 			)
 		)
-		(property "Footprint" "Capacitor_SMD:CP_Elec_10x10.5"
+		(property "Footprint" "Capacitor_SMD:C_0603_1608Metric"
 			(at 141.9352 66.04 0)
 			(hide yes)

Commit message: A bunch of schematic changes
Parts:
- added J17: Guitar input, SSK02-FPH-254-A2:SAMESKY_SSK02-FPH-254-A2, symbol female_headers_2pin:SSK02-FPH-254-A2
Connections:
- net GND: now also J17.1
- net Guitar_In: now also J17.2

Commit message: First iteration, need to tweak some things
Parts:
- added C2, C35, C38, C39: 10uF, Capacitor_SMD:C_1206_3216Metric, symbol Device:C_Small
- added C32, C36, C37, C40: .1uF, Capacitor_SMD:C_0402_1005Metric_Pad0.74x0.62mm_HandSolder, symbol Device:C_Small
- added unit 3 of U6
- added unit 2 of U6
- added unit 3 of U7
- J17: footprint SSK02-FPH-254-A2:SAMESKY_SSK02-FPH-254-A2 -> header_fem_pin2:SAMESKY_SSK02-FPH-254-A2
- renumbered U8 to U7
Connections:
- net +9V: now also C37.1, C38.2, C39.1, C40.2, U6.8 (V+), U7.8 (V+)
- net -9V: now also C2.2, C32.2, C35.1, C36.1, U6.4 (V-), U7.4 (V-)
- net GND: now also TP3.1, C2.1, C32.1, C35.2, C36.2, C37.2, C38.1, C39.2, C40.1, U6.5 (+)
- net GuitarIn: now also C7.1, D2.3 (COM), R5.2, R6.1, TP2.1
- net Guitar_In: now also TP1.1
- net at D2.2 (K), U7.1, U7.2 (-): no longer TP1.1
- net at C9.2, R7.2, R8.1: now also U7.5 (+); no longer U7.3 (+)
- new net: D2.1 (A), U7.6 (-), U7.7
- new net: U6.6 (-), U6.7
Other:
- note added: "Op-amp rails, caps will prevent ringing and match impedances (the trace is inductive) of the longer trace."
- moved on the sheet: TP1

Commit message: Changes Luke caught
Parts:
- removed TP4: TestPoint, TestPoint:TestPoint_Loop_D2.50mm_Drill1.85mm, symbol Connector:TestPoint
Connections:
- net +9V: now also R10.2; no longer R9.2
- net GND: now also R9.1; no longer R10.1
- net at C8.2, U7.3 (+): now also R10.1, R9.2; no longer R10.2, R9.1
Other:
- moved on the sheet: R10, R9
Changed lines of the file:
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@@
 	)
 	(junction
+		(at 134.62 68.58)
+		(diameter 0)
+		(color 0 0 0 0)
+	)
+	(junction
 		(at 142.24 93.98)
 		(diameter 0)
@@
 	)
 	(junction
+		(at 134.62 57.15)
+		(diameter 0)
+		(color 0 0 0 0)
+	)
+	(junction
 		(at 251.46 54.61)
 		(diameter 0)
@@
 	)
 	(junction
-		(at 134.62 57.15)
-		(diameter 0)
-		(color 0 0 0 0)
-	)
-	(junction
 		(at 140.97 121.92)
 		(diameter 0)
@@
 	)
 	(junction
-		(at 134.62 68.58)
-		(diameter 0)
-		(color 0 0 0 0)
-	)
-	(junction
 		(at 251.46 31.75)
 		(diameter 0)
@@
 	(wire
 		(pts
+			(xy 134.62 66.04) (xy 134.62 68.58)
+		)
+		(stroke
+			(width 0)
+			(type default)
+		)
+	)
+	(wire
+		(pts
 			(xy 140.97 68.58) (xy 153.67 68.58)
 		)
@@
 	(wire
 		(pts
-			(xy 134.62 68.58) (xy 140.97 68.58)
+			(xy 251.46 34.29) (xy 251.46 31.75)
 		)
 		(stroke
@@
 	(wire
 		(pts
-			(xy 251.46 34.29) (xy 251.46 31.75)
+			(xy 153.67 63.5) (xy 147.32 63.5)
 		)
 		(stroke
@@
 	(wire
 		(pts
-			(xy 153.67 63.5) (xy 147.32 63.5)
+			(xy 78.74 85.09) (xy 95.25 85.09)
 		)
 		(stroke
@@
 	(wire
 		(pts
-			(xy 78.74 85.09) (xy 95.25 85.09)
+			(xy 147.32 63.5) (xy 147.32 55.88)
 		)
 		(stroke
@@
 	(wire
 		(pts
-			(xy 147.32 63.5) (xy 147.32 55.88)
+			(xy 134.62 121.92) (xy 134.62 123.19)
 		)
 		(stroke
@@
 	(wire
 		(pts
-			(xy 134.62 121.92) (xy 134.62 123.19)
+			(xy 134.62 57.15) (xy 134.62 58.42)
 		)
 		(stroke
@@
 	(wire
 		(pts
-			(xy 134.62 57.15) (xy 134.62 59.69)
-		)
-		(stroke
-			(width 0)
-			(type default)
-		)
-	)
-	(wire
-		(pts
 			(xy 78.74 76.2) (xy 78.74 74.93)
 		)
@@
 	(wire
 		(pts
+			(xy 134.62 68.58) (xy 140.97 68.58)
+		)
+		(stroke
+			(width 0)
+			(type default)
+		)
+	)
+	(wire
+		(pts
 			(xy 71.12 96.52) (xy 73.66 96.52)
 		)
@@
 	(wire
 		(pts
-			(xy 134.62 67.31) (xy 134.62 68.58)
+			(xy 168.91 55.88) (xy 168.91 66.04)
 		)
 		(stroke
@@
 	(wire
 		(pts
-			(xy 168.91 55.88) (xy 168.91 66.04)
+			(xy 134.62 68.58) (xy 134.62 71.12)
 		)
 		(stroke
@@
 	(wire
 		(pts
-			(xy 134.62 68.58) (xy 134.62 71.12)
-		)
-		(stroke
-			(width 0)
-			(type default)
-		)
-	)
-	(wire
-		(pts
 			(xy 203.2 81.28) (xy 203.2 78.74)
 		)
@@
 	(symbol
 		(lib_id "Device:R_US")
-		(at 134.62 74.93 180)
+		(at 134.62 62.23 180)
 		(unit 1)
 		(body_style 1)
@@
 		(in_pos_files yes)
 		(dnp no)
-		(fields_autoplaced yes)
 		(property "Reference" "R10"
-			(at 137.16 73.6599 0)
+			(at 128.27 60.452 0)
 			(show_name no)
 			(do_not_autoplace no)
@@
 		)
 		(property "Value" "620k"
-			(at 137.16 76.1999 0)
+			(at 128.524 63.5 0)
 			(show_name no)
 			(do_not_autoplace no)
@@
 		)
 		(property "Footprint" "Resistor_SMD:R_1206_3216Metric"
-			(at 133.604 74.676 90)
+			(at 133.604 61.976 90)
 			(hide yes)
 			(show_name no)
@@
 		)
 		(property "Datasheet" ""
-			(at 134.62 74.93 0)
+			(at 134.62 62.23 0)
 			(hide yes)
 			(show_name no)
@@
 		)
 		(property "Description" "Resistor, US symbol"
-			(at 134.62 74.93 0)
+			(at 134.62 62.23 0)
 			(hide yes)
 			(show_name no)
@@
 	(symbol
 		(lib_id "Device:R_US")
-		(at 134.62 63.5 180)
+		(at 134.62 74.93 180)
 		(unit 1)
 		(body_style 1)
@@
 		(dnp no)
 		(property "Reference" "R9"
-			(at 126.746 62.23 0)
+			(at 126.746 73.66 0)
 			(show_name no)
 			(do_not_autoplace no)
@@
 		)
 		(property "Value" "100k"
-			(at 126.746 64.77 0)
+			(at 126.746 76.2 0)
 			(show_name no)
 			(do_not_autoplace no)
@@
 		)
 		(property "Footprint" "Resistor_SMD:R_1206_3216Metric"
-			(at 133.604 63.246 90)
+			(at 133.604 74.676 90)
 			(hide yes)
 			(show_name no)
@@
 		)
 		(property "Datasheet" ""
-			(at 134.62 63.5 0)
+			(at 134.62 74.93 0)
 			(hide yes)
 			(show_name no)
@@
 		)
 		(property "Description" "Resistor, US symbol"
-			(at 134.62 63.5 0)
+			(at 134.62 74.93 0)
 			(hide yes)
 			(show_name no)
@@
 					(unit 1)
 				)
-			)
-		)
-	)
-	(symbol
-		(lib_id "Connector:TestPoint")
-		(at 106.68 93.98 180)
-		(unit 1)
-		(body_style 1)
-		(exclude_from_sim no)
-		(in_bom yes)
-		(on_board yes)
-		(in_pos_files yes)
-		(dnp no)
-		(fields_autoplaced yes)
-		(property "Reference" "TP4"
-			(at 109.22 96.0119 0)
-			(show_name no)
-			(do_not_autoplace no)
-			(effects
-				(font
-					(size 1.27 1.27)
-				)
-				(justify right)
-			)
-		)
-		(property "Value" "TestPoint"
-			(at 109.22 98.5519 0)
-			(show_name no)
-			(do_not_autoplace no)
-			(effects
-				(font
-					(size 1.27 1.27)
-				)
-				(justify right)
-			)
-		)
-		(property "Footprint" "TestPoint:TestPoint_Loop_D2.50mm_Drill1.85mm"
-			(at 101.6 93.98 0)
-			(hide yes)
-			(show_name no)
-			(do_not_autoplace no)
-			(effects
-				(font
-					(size 1.27 1.27)
-				)
-			)
-		)
-		(property "Datasheet" ""
-			(at 101.6 93.98 0)
-			(hide yes)
-			(show_name no)
-			(do_not_autoplace no)
-			(effects
-				(font
-					(size 1.27 1.27)
-				)
-			)
-		)
-		(property "Description" "test point"
-			(at 106.68 93.98 0)
-			(hide yes)
-			(show_name no)
-			(do_not_autoplace no)
-			(effects
-				(font
-					(size 1.27 1.27)
-				)
-			)
-		)
-		(pin "1"
-		)
-		(instances
-			(project "rpi_and_peripherals"
-				(path "/149bebb8-d22c-435a-adf0-1313d3be5660/482e9c29-4e2a-4660-9574-25cec0041a8a"
-					(reference "TP4")
-					(unit 1)
-				)
-			)
-			(project "KiCad"
-				(path "/24850b4e-1ce6-41a1-b1f6-c45749a7c3af/482e9c29-4e2a-4660-9574-25cec0041a8a"
-					(reference "TP4")
-					(unit 1)
-				)
