File: KiCad/analogFE.kicad_sch (KiCad schematic)
At the start: 31 parts, among them J17 Guitar input, U6 NE5532, U7 NE5532

Commit message: Changes to the BoM
Parts:
- C10, C11: Part_Number (none) -> C0603C100J5GACTU
- C2, C35, C38, C39: Part_Number (none) -> GMC31X7R106K50NT
- C32, C36, C37, C40: Part_Number (none) -> GRM155R71H104KE14D
- C6: Part_Number (none) -> C0603C104K5RACTU
- C7: Part_Number (none) -> CL10B333KC8WPNC
- C8, C9: Part_Number (none) -> C0603C105K4RACTU
- J17: Part_Number (none) -> SSK02-FPH-254-A2
- R1: Part_Number (none) -> KTR18EZPF1004
- R10, R8: Part_Number (none) -> ERJ-8ENF6653V
- R2: Part_Number (none) -> CR1206-JW-223ELF
- R3: Part_Number (none) -> ERA-8AEB473V
- R4, R6, R7, R9: Part_Number (none) -> RC1206FR-07100KL
- R5: Part_Number (none) -> RK73H2BTTD4700F
- U6, U7: Part_Number (none) -> NE5532DR
