File: KiCad/KiCad.kicad_pcb (KiCad board)
At the start: 2 copper layers, 234.5 x 128.4 mm, 8 parts, among them U3 PCM5102A, U5 PCM1808-Q1_PW_14

Commit message: Changed footprints, added powersystem
Parts:
- added BT1: 9V, Battery:BatteryHolder_MPD_BA9VPC_1xPP3, F.Cu at (119.9, 53.3)
- added C10: 10pF, Capacitor_SMD:CP_Elec_5x4.5, F.Cu at (127.0, 107.3)
- added C11: 10pF, Capacitor_SMD:CP_Elec_5x4.5, F.Cu at (127.0, 114.1)
- added C12: 2.2nF, Capacitor_SMD:C_0402_1005Metric, F.Cu at (165.6, 112.8)
- added C13: 2.2nF, Capacitor_SMD:C_0402_1005Metric, F.Cu at (165.6, 114.8)
- added C14: 2.2uF, Capacitor_SMD:C_0603_1608Metric, F.Cu at (166.1, 91.4)
- added C15: 0.1uF, Capacitor_SMD:C_0603_1608Metric, F.Cu at (166.1, 93.9)
- added C16: 0.1uF, Capacitor_SMD:C_0603_1608Metric, F.Cu at (166.1, 96.4)
- added C17: 0.1uF, Capacitor_SMD:C_0603_1608Metric, F.Cu at (166.1, 99.0)
- added C18: 0.1uF, Capacitor_SMD:C_0603_1608Metric, F.Cu at (166.1, 101.5)
- added C19: 10uF, Capacitor_SMD:CP_Elec_6.3x5.4, F.Cu at (158.8, 94.2)
- added C20: 10uF, Capacitor_SMD:CP_Elec_6.3x5.4, F.Cu at (158.8, 102.4)
- added C21: 10uF, Capacitor_SMD:CP_Elec_6.3x5.4, F.Cu at (158.8, 110.5)
- added C22: 10uF, Capacitor_SMD:CP_Elec_6.3x5.4, F.Cu at (158.8, 118.7)
- added C23: 2.2uF, Capacitor_SMD:C_0603_1608Metric, F.Cu at (166.1, 104.0)
- added C24: 10uF, Capacitor_SMD:CP_Elec_6.3x5.4, F.Cu at (130.0, 80.5)
- added C25: 100uF, Capacitor_SMD:C_Elec_6.3x7.7, F.Cu at (140.3, 80.5)
- added C26: 1uF, Capacitor_SMD:CP_Elec_4x5.7, F.Cu at (120.8, 79.4)
- added C27: 1uF, Capacitor_SMD:CP_Elec_4x5.7, F.Cu at (120.8, 85.2)
- added C6: 0.1uF, Capacitor_SMD:CP_Elec_5x4.5, F.Cu at (127.0, 93.6)
- added C7: 33nF, Capacitor_SMD:CP_Elec_5x4.5, F.Cu at (127.0, 100.4)
- added C8: 1mF, Capacitor_SMD:CP_Elec_10x10.5, F.Cu at (138.9, 96.2)
- added C9: 1mF, Capacitor_SMD:CP_Elec_10x10.5, F.Cu at (138.9, 108.2)
- added D1: BAT54ADW, Package_TO_SOT_SMD:SOT-363_SC-70-6, F.Cu at (141.3, 116.1)
- added R1: 1M, Resistor_SMD:R_1206_3216Metric, F.Cu at (119.7, 91.8)
- added R10: 620k, Resistor_SMD:R_1206_3216Metric, F.Cu at (119.7, 121.6)
- added R11: 470, Resistor_SMD:R_1206_3216Metric, F.Cu at (166.9, 106.9)
- added R12: 470, Resistor_SMD:R_1206_3216Metric, F.Cu at (166.9, 110.2)
- added R2: 22k, Resistor_SMD:R_1206_3216Metric, F.Cu at (119.7, 95.1)
- added R3: 47k, Resistor_SMD:R_1206_3216Metric, F.Cu at (119.7, 98.4)
- added R4: 100k, Resistor_SMD:R_1206_3216Metric, F.Cu at (119.7, 101.8)
- added R5: 470, Resistor_SMD:R_1206_3216Metric, F.Cu at (119.7, 105.1)
- added R6: 100k, Resistor_SMD:R_1206_3216Metric, F.Cu at (119.7, 108.4)
- added R7: 100k, Resistor_SMD:R_1206_3216Metric, F.Cu at (119.7, 111.7)
- added R8: 620k, Resistor_SMD:R_1206_3216Metric, F.Cu at (119.7, 115.0)
- added R9: 100k, Resistor_SMD:R_1206_3216Metric, F.Cu at (119.7, 118.3)
- added TP1: TestPoint, TestPoint:TestPoint_Loop_D2.50mm_Drill1.85mm, F.Cu at (148.8, 92.9)
- added TP2: TestPoint, TestPoint:TestPoint_Loop_D2.50mm_Drill1.85mm, F.Cu at (148.8, 98.3)
- added TP3: TestPoint, TestPoint:TestPoint_Loop_D2.50mm_Drill1.85mm, F.Cu at (148.8, 103.8)
- added TP4: TestPoint, TestPoint:TestPoint_Loop_D2.50mm_Drill1.85mm, F.Cu at (148.8, 109.2)
- added U7: NE5532, op_amp:D8-L, F.Cu at (135.4, 117.5)
- added U8: NE5532, op_amp:D8-L, F.Cu at (135.4, 123.9)
- added U9: PCM5102APW, Package_SO:Texas_PW0020A_TSSOP-20_4.4x6.5mm_P0.65mm, F.Cu at (106.3, 58.9)
- C1, C2: footprint Capacitor_SMD:C_0603_1608Metric -> Capacitor_SMD:CP_Elec_4x5.7
- C3, C4: value 0.1uF/10uF -> 0.1uF; footprint Capacitor_SMD:C_0805_2012Metric -> Capacitor_SMD:C_0603_1608Metric
- C5: value 0.1uF/10uF -> 10uF; footprint Capacitor_SMD:C_0805_2012Metric -> Capacitor_SMD:CP_Elec_6.3x5.4
- U3: value PCM5102A -> LT1054; footprint Package_SO:TSSOP-20_4.4x6.5mm_P0.65mm -> charge_pump:SOIC127P1030X265-16N
- moved C3 88.0 mm to (81.1, 111.1)
- moved C4 86.5 mm to (81.1, 113.6)
- moved C2 78.4 mm to (83.0, 106.9)
- moved C1 76.9 mm to (83.0, 101.1)
- moved U5 65.9 mm to (91.3, 109.7)
- moved C5 63.4 mm to (92.2, 102.2)
- moved U3 43.8 mm to (108.5, 49.0)
- moved U2 37.4 mm to (99.2, 46.1)
Connections:
- C3 pad 2: GND -> +9V
- C4 pad 2: GND -> +9V
- C5 pad 2: GND -> +9V
- U2 pad 36: PICO_DEBUG -> unconnected-(U2-3V3(OUT)-Pad36)
- U2 pad 38: GND -> +9V
- U2 pad 8: GND -> +9V
- U3 pad 1: +3V3 -> unconnected-(U3-FB/SHDN-Pad1)
- U3 pad 10: GND -> (no net)
- U3 pad 11: GND -> (no net)
- U3 pad 12: MCK -> (no net)
- U3 pad 13: BCK -> (no net)
- U3 pad 14: DAC Dout -> (no net)
- U3 pad 15: LRCK -> (no net)
- U3 pad 16: GND -> (no net)
- U3 pad 2: unconnected-(U3-CAPP-Pad2) -> Net-(U3-CAP+)
- U3 pad 3: GND -> +9V
- U3 pad 4: unconnected-(U3-CAPM-Pad4) -> Net-(U3-CAP+)
- U3 pad 5: -3V3 -> +9V
- U3 pad 6: Net-(U3-OUTL) -> unconnected-(U3-VREF-Pad6)
- U3 pad 7: Net-(U3-OUTR) -> unconnected-(U3-OSC-Pad7)
- U3 pad 8: +3V3 -> +9V
- U3 pad 9: GND -> (no net)
- U5 pad 10: GND -> +9V
- U5 pad 11: GND -> +9V
- U5 pad 12: GND -> +9V
- U5 pad 2: GND -> +9V
- U5 pad 5: GND -> +9V
Routing:
- net GND: track 111.4 -> 0.00 mm, vias 2 -> 0
- net LRCK: track 76.9 -> 0.00 mm, vias 2 -> 0
- net BCK: track 64.6 -> 0.00 mm, vias 2 -> 0
- net DAC Dout: track 58.7 -> 0.00 mm, vias 1 -> 0
- net MCK: track 53.9 -> 0.00 mm
- net +3V3: track 50.5 -> 0.00 mm, vias 4 -> 0
- net ADC Din: track 48.5 -> 0.00 mm, vias 1 -> 0
- net +5V: track 23.1 -> 0.00 mm, vias 2 -> 0
- net Net-(U5-VREF): track 12.1 -> 0.00 mm, vias 2 -> 0
- net Net-(U5-VINR): track 2.97 -> 0.00 mm
- net Net-(U5-VINL): track 2.92 -> 0.00 mm

Commit message: Updates for 10_18_26
Parts:
- moved R12 137.5 mm to (34.0, 75.0)
- moved R11 137.3 mm to (34.0, 72.5)
- moved C14 136.7 mm to (33.7, 57.5)
- moved C15 136.7 mm to (33.7, 60.0)
- moved C16 136.7 mm to (33.7, 62.5)
- moved C17 136.7 mm to (33.7, 65.0)
- moved C18 136.7 mm to (33.7, 67.5)
- moved C23 136.7 mm to (33.7, 70.0)
- moved C12 136.7 mm to (33.2, 78.9)
- moved C13 136.7 mm to (33.2, 80.8)
- moved D1 118.6 mm to (37.8, 58.1)
- moved BT1 111.9 mm to (29.0, 118.5)
- moved TP1 103.2 mm to (51.1, 59.5), turned to 90 degrees
- moved TP2 100.1 mm to (56.5, 59.5), turned to 90 degrees
- moved TP3 97.4 mm to (62.0, 59.5), turned to 90 degrees
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Other:
- board size 234.5 x 128.4 mm -> 58.9 x 90 mm

Commit message: Pushing PCB, and controls schem
Parts:
- removed D1: BAT54ADW, Package_TO_SOT_SMD:SOT-363_SC-70-6
- removed U2: ~, rpi_foot:rpi_dev_foot
- removed U3: LT1054, charge_pump:SOIC127P1030X265-16N
- added A1: RaspberryPi_Pico, Module:RaspberryPi_Pico_Common_Unspecified, F.Cu at (196.8, 102.0)
- added C28: 1uF, Capacitor_SMD:C_0603_1608Metric, F.Cu at (169.0, 132.1)
- added C29: 1uF, Capacitor_SMD:C_0603_1608Metric, F.Cu at (157.2, 121.9)
- added C30: 1uF, Capacitor_SMD:C_0603_1608Metric, F.Cu at (129.3, 117.6)
- added C31: 1uF, Capacitor_SMD:C_0603_1608Metric, F.Cu at (145.2, 134.8)
- added C32: 1uF, Capacitor_SMD:C_0603_1608Metric, F.Cu at (145.2, 137.3)
- added C33: 1uF, Capacitor_SMD:C_0603_1608Metric, F.Cu at (145.2, 139.8)
- added C34: 1uF, Capacitor_SMD:C_0603_1608Metric, F.Cu at (145.2, 142.3)
- added C35: 1uF, Capacitor_SMD:C_0603_1608Metric, F.Cu at (145.2, 144.8)
- added D2: BAT54S, Package_TO_SOT_SMD:SOT-23, F.Cu at (209.5, 77.1)
- added R13: 0, Resistor_SMD:R_0603_1608Metric, F.Cu at (187.5, 77.1)
- added R14: 0, Resistor_SMD:R_0603_1608Metric, F.Cu at (192.7, 79.4)
- added U1: LT1054, charge_pump:SOIC127P1030X265-16N, F.Cu at (240.4, 124.9)
- added U12: MCP1703T-3302E/DB, lin_reg:SOT-223_3MC_MCH, F.Cu at (161.6, 131.7)
- added U13: MCP1703T-5002E/DB, lin_reg_50:SOT-223_3MC_MCH, F.Cu at (164.6, 123.9)
- added U14: MCP1703T-5002E/DB, lin_reg_50:SOT-223_3MC_MCH, F.Cu at (147.2, 129.9)
- added U15: MCP1703T-3302E/DB, lin_reg:SOT-223_3MC_MCH, F.Cu at (136.5, 126.7)
- added U6: NE5532, op_amp:D8-L, F.Cu at (232.2, 72.6)
- moved C11 218.8 mm to (270.7, 71.8)
- moved C10 206.6 mm to (259.0, 73.0)
- moved R1 205.1 mm to (244.8, 72.6), turned to 90 degrees
- moved R2 194.3 mm to (233.8, 79.7), turned to 90 degrees
- moved R3 191.4 mm to (231.1, 79.8), turned to 90 degrees
- moved R4 187.0 mm to (226.9, 78.4), turned to 180 degrees
- moved C6 186.5 mm to (239.2, 76.5), turned to 180 degrees
- moved R5 181.4 mm to (221.4, 78.4), turned to 180 degrees
- moved R7 177.0 mm to (209.7, 66.7), turned to 180 degrees
- moved R6 172.9 mm to (212.8, 75.6), turned to 90 degrees
- moved R10 172.5 mm to (211.9, 82.1), turned to 180 degrees
- moved R9 172.1 mm to (212.0, 85.5)
- moved R8 172.0 mm to (204.3, 66.7), turned to 180 degrees
- moved C7 164.6 mm to (217.3, 74.0), turned to 90 degrees
- moved U5 144.9 mm to (179.6, 80.7)
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Connections:
- net Net-(C12-Pad1) renamed SIG_R_OUT
- net Net-(C13-Pad1) renamed SIG_L_OUT
- C1 pad 1: Net-(U5-VINR) -> Net-(C1-Pad1)
- C1 pad 2: /pcm_1808/R-ch IN -> Net-(D2-COM)
- C12 pad 2: +9V -> GNDA
- C13 pad 2: +9V -> GNDA
- C15 pad 1: +3V3 -> +3.3VA
- C15 pad 2: +9V -> GNDA
- C16 pad 1: +3V3 -> +3.3VA
- C16 pad 2: +9V -> GNDA
- C19 pad 1: +3V3 -> +3.3VA
- C19 pad 2: +9V -> GNDA
- C2 pad 1: Net-(U5-VINL) -> Net-(C2-Pad1)
- C2 pad 2: /pcm_1808/L-ch IN -> Net-(D2-COM)
- C20 pad 1: +3V3 -> +3.3VA
- C20 pad 2: +9V -> GNDA
- C23 pad 1: -3V3 -> Net-(C23-Pad1)
- C23 pad 2: +9V -> GNDA
- C4 pad 1: +5V -> GNDA
- C4 pad 2: +9V -> +5VA
- C7 pad 1: Net-(D1A-A) -> Net-(D2-COM)
- R5 pad 2: Net-(D1A-A) -> Net-(D2-COM)
- R6 pad 1: Net-(D1A-A) -> Net-(D2-COM)
- TP2 pad 1: Net-(D1A-A) -> Net-(D2-COM)
- U5 pad 2: +9V -> GNDA
- U5 pad 3: +5V -> +5VA
- U9 pad 1: +3V3 -> +3.3VA
- U9 pad 18: unconnected-(U9-LDOO-Pad18) -> Net-(C18-Pad1)
- U9 pad 5: -3V3 -> unconnected-(U9-VNEG-Pad5)
- U9 pad 8: +3V3 -> +3.3VA
Routing:
- net GNDA: track 0.00 -> 49.1 mm
- net MCK: track 0.00 -> 43.5 mm, vias 0 -> 2
- net BCK: track 0.00 -> 41.0 mm, vias 0 -> 1
- net LRCK: track 0.00 -> 39.6 mm, vias 0 -> 2
- net Net-(D2-COM): track 0.00 -> 30.4 mm
- net ADC Din: track 0.00 -> 16.9 mm, vias 0 -> 1
- net Net-(C18-Pad1): track 0.00 -> 11.5 mm
- net Net-(U8A-+): track 0.00 -> 11.3 mm
- net Net-(U7A-+): track 0.00 -> 10.7 mm
- net Net-(U5-VINL): track 0.00 -> 10.3 mm
- net Net-(R4-Pad2): track 0.00 -> 9.64 mm
- net +9V: track 0.00 -> 8.54 mm
- net +5VA: track 0.00 -> 7.96 mm
- net Net-(C1-Pad1): track 0.00 -> 7.91 mm
- net Net-(D2-A): track 0.00 -> 7.81 mm
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Other:
- board outline removed
- board text added: "sigout"

Commit message: Preparing to auto-route
Parts:
- removed U9: PCM5102APW, Package_SO:Texas_PW0020A_TSSOP-20_4.4x6.5mm_P0.65mm
- moved U15 29.2 mm to (156.3, 148.3), turned to 180 degrees
- moved C29 27.4 mm to (149.4, 148.1)
- moved C32 26.1 mm to (129.7, 158.2)
- moved C34 26.1 mm to (129.7, 163.3)
- moved C35 26.1 mm to (129.7, 165.8)
- moved C33 26.1 mm to (129.7, 160.8)
- moved C10 21.9 mm to (248.9, 53.5), turned to 90 degrees
- moved C11 21.9 mm to (260.6, 52.4)
- moved U6 9.41 mm to (222.8, 72.5)
- moved U12 9.18 mm to (156.2, 139.1), turned to 180 degrees
- moved U14 9.01 mm to (156.2, 130.3), turned to 180 degrees
- moved U13 8.69 mm to (156.3, 121.4), turned to 180 degrees
- moved C31 6.10 mm to (148.4, 140.0)
- moved R2 5.97 mm to (228.0, 81.3)
- moved R14 5.85 mm to (186.9, 80.2)
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Connections:
- BT1 pad 2: +9V -> GND
- C1 pad 2: Net-(D2-COM) -> /pcm_1808/R-ch IN
- C10 pad 2: +9V -> GND
- C11 pad 1: +9V -> GND
- C11 pad 2: +9V -> -9V
- C17 pad 2: +9V -> GND
- C18 pad 2: +9V -> GND
- C2 pad 2: Net-(D2-COM) -> /pcm_1808/L-ch IN
- C21 pad 2: +9V -> GND
- C22 pad 2: +9V -> GND
- C25 pad 1: +9V -> GND
- C25 pad 2: +9V -> -9V
- C26 pad 2: +9V -> GND
- C27 pad 2: +9V -> GND
- C28 pad 2: +9V -> GND
- C29 pad 2: +9V -> GND
- C3 pad 2: +9V -> GND
- C30 pad 2: +9V -> GND
- C31 pad 2: +9V -> GND
- C32 pad 2: +9V -> GND
- C33 pad 2: +9V -> GND
- C34 pad 2: +9V -> GND
- C35 pad 2: +9V -> GND
- C5 pad 2: +9V -> GND
- C7 pad 2: +9V -> GND
- C9 pad 1: +9V -> GND
- R1 pad 2: +9V -> GND
- R10 pad 1: +9V -> GND
- R2 pad 1: +9V -> GND
- R3 pad 1: +9V -> GND
- R6 pad 2: +9V -> GND
- R7 pad 1: +9V -> GND
- R8 pad 2: +9V -> -9V
- U1 pad 3: +9V -> GND
- U1 pad 5: +9V -> -9V
- U12 pad 2: +9V -> GND
- U13 pad 2: +9V -> GND
- U14 pad 2: +9V -> GND
- U15 pad 2: +9V -> GND
- U5 pad 10: +9V -> GND
- U5 pad 11: +9V -> GND
- U5 pad 12: +9V -> GND
- U5 pad 5: +9V -> GND
Routing:
- net Net-(U7A-+): track 10.7 -> 0.14 mm
- net Net-(U5-VINL): track 10.3 -> 0.00 mm
- net +9V: track 8.54 -> 18.3 mm
- net GND: track 0.00 -> 8.54 mm
- net Net-(U6A--): track 6.69 -> 12.5 mm
- net Net-(U6A-+): track 6.79 -> 12.2 mm
- net Net-(D2-K): track 5.43 -> 1.00 mm
- net Net-(C1-Pad1): track 7.91 -> 3.54 mm
- net Net-(U5-VINR): track 5.01 -> 2.36 mm
- net Net-(R4-Pad2): track 9.64 -> 7.17 mm
- net Net-(C2-Pad1): track 2.72 -> 3.86 mm

Commit message: PCB ex
Parts:
- removed BT1: 9V, Battery:BatteryHolder_MPD_BA9VPC_1xPP3
- removed C10, C11: 10pF, Capacitor_SMD:CP_Elec_5x4.5
- removed C30, C32, C33: 1uF, Capacitor_SMD:C_0603_1608Metric
- removed C8, C9: 1mF, Capacitor_SMD:CP_Elec_10x10.5
- removed TP1, TP2, TP3, TP4: TestPoint, TestPoint:TestPoint_Loop_D2.50mm_Drill1.85mm
- added IN1: SAMESKY_SSK02-FPH-254-A2, header_fem:SAMESKY_SSK02-FPH-254-A2, F.Cu at (237.6, 78.9)
- added SW2: SAMESKY_SSK02-FPH-254-A3, header_fem_3pin:SAMESKY_SSK02-FPH-254-A3, F.Cu at (193.3, 88.0)
- added SW3: SAMESKY_SSK02-FPH-254-A3, header_fem_3pin:SAMESKY_SSK02-FPH-254-A3, F.Cu at (167.9, 99.9)
- added SW4: SAMESKY_SSK02-FPH-254-A3, header_fem_3pin:SAMESKY_SSK02-FPH-254-A3, F.Cu at (186.1, 115.6)
- added SW5: SAMESKY_SSK02-FPH-254-A2, header_fem:SAMESKY_SSK02-FPH-254-A2, F.Cu at (216.7, 86.8)
- added SW6: SAMESKY_SSK02-FPH-254-A2, header_fem:SAMESKY_SSK02-FPH-254-A2, F.Cu at (220.0, 86.8)
- added U10: PCM5102APW, Package_SO:Texas_PW0020A_TSSOP-20_4.4x6.5mm_P0.65mm, F.Cu at (162.2, 96.5)
- moved C26 167.6 mm to (224.0, 119.7)
- moved C27 162.2 mm to (224.0, 124.7)
- moved C25 158.8 mm to (203.7, 127.9)
- moved C24 157.6 mm to (205.6, 119.2), turned to 90 degrees
- moved C22 76.3 mm to (158.0, 86.0), turned to 90 degrees
- moved C34 72.8 mm to (192.1, 126.0)
- moved C35 66.5 mm to (183.1, 126.2)
- moved U15 47.1 mm to (194.9, 121.4), turned to -90 degrees
- moved U12 34.3 mm to (185.6, 121.5), turned to -90 degrees
- moved C31 29.2 mm to (174.1, 126.2)
- moved C29 27.3 mm to (165.4, 126.0), turned to 0 degrees
- moved U1 25.8 mm to (214.8, 121.4), turned to 90 degrees
- moved C17 25.1 mm to (153.0, 87.3), turned to 90 degrees
- moved U14 22.4 mm to (176.6, 121.3), turned to -90 degrees
- moved C28 19.1 mm to (179.9, 116.5), turned to 0 degrees
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Connections:
- C12 pad 2: GNDA -> GND
- C13 pad 2: GNDA -> GND
- C15 pad 2: GNDA -> GND
- C16 pad 2: GNDA -> GND
- C19 pad 2: GNDA -> GND
- C2 pad 2: /pcm_1808/L-ch IN -> /pcm_1808/R-ch IN
- C20 pad 2: GNDA -> GND
- C23 pad 2: GNDA -> GND
- C4 pad 1: GNDA -> GND
- D2 pad 3: Net-(D2-COM) -> /pcm_1808/R-ch IN
- U5 pad 2: GNDA -> GND
- U7 pad 4: (no net) -> -9V
- U7 pad 8: (no net) -> +9V
- U8 pad 8: (no net) -> +9V
Routing:
- net -9V: track 0.00 -> 153.0 mm, vias 0 -> 4
- net +5VA: track 7.96 -> 106.0 mm, vias 0 -> 2
- net +9V: track 18.3 -> 115.8 mm, vias 0 -> 4
- net GNDA: track 49.1 -> 0.00 mm
- net +3V3: track 5.07 -> 43.5 mm, vias 0 -> 2
- net +3.3VA: track 2.96 -> 32.4 mm, vias 0 -> 2
- net GND: track 8.54 -> 35.2 mm, vias 0 -> 26
- net LRCK: track 39.6 -> 15.9 mm, vias 2 -> 0
- net DAC Dout: track 0.17 -> 22.9 mm, vias 0 -> 2
- net Net-(D2-COM): track 30.5 -> 10.8 mm
- net /pcm_1808/R-ch IN: track 0.00 -> 17.0 mm
- net Net-(U1-CAP-): track 0.00 -> 16.4 mm
- net unconnected-(A1-GPIO16-Pad21)_1: track 0.00 -> 15.2 mm
- net Net-(U1-CAP+): track 0.00 -> 11.5 mm
- net unconnected-(A1-GPIO17-Pad22)_1: track 0.00 -> 11.1 mm
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- added copper zone on B.Cu, net GND
- added copper zone on F.Cu, net GND
Other:
- board text removed: "sigout"
