File: KiCad/KiCad.kicad_pcb (KiCad board)
At the start: 2 copper layers, 66 parts, among them U1 LT1054, U12 MCP1703T-3302E/DB, U13 MCP1703T-5002E/DB, U14 MCP1703T-5002E/DB, U15 MCP1703T-3302E/DB, U5 PCM1808-Q1_PW_14, U6 NE5532, U7 NE5532, U8 NE5532, U9 PCM5102APW

Commit message: Best one yet
Parts:
- removed BT1: 9V, Battery:BatteryHolder_MPD_BA9VPC_1xPP3
- removed TP1, TP2, TP3, TP4: TestPoint, TestPoint:TestPoint_Loop_D2.50mm_Drill1.85mm
- removed U8: NE5532, op_amp:D8-L
- removed U9: PCM5102APW, Package_SO:Texas_PW0020A_TSSOP-20_4.4x6.5mm_P0.65mm
- added J1: SSK02-FPH-254-A2, header_female_2pin:SAMESKY_SSK02-FPH-254-A2, F.Cu at (235.4, 123.1)
- added J10: Battery in, header_female_2pin:SAMESKY_SSK02-FPH-254-A2, F.Cu at (195.0, 127.3)
- added J11: P_Switch, header_female_2pin:SAMESKY_SSK02-FPH-254-A2, F.Cu at (204.5, 128.1)
- added J2: SSK02-FPH-254-A3, header_female_3pin:SAMESKY_SSK02-FPH-254-A3, F.Cu at (225.6, 91.8)
- added J3: SSK02-FPH-254-A3, header_female_3pin:SAMESKY_SSK02-FPH-254-A3, F.Cu at (198.2, 105.4)
- added J4: SSK02-FPH-254-A3, header_female_3pin:SAMESKY_SSK02-FPH-254-A3, F.Cu at (207.4, 121.7)
- added J5: SSK02-FPH-254-A2, header_female_2pin:SAMESKY_SSK02-FPH-254-A2, F.Cu at (250.6, 92.5)
- added J6: SSK02-FPH-254-A2, header_female_2pin:SAMESKY_SSK02-FPH-254-A2, F.Cu at (247.6, 92.5)
- added J7: SSK02-FPH-254-A2, header_female_2pin:SAMESKY_SSK02-FPH-254-A2, F.Cu at (236.7, 94.5)
- added J8: SSK02-FPH-254-A2, header_female_2pin:SAMESKY_SSK02-FPH-254-A2, F.Cu at (240.4, 123.0)
- added J9: SSK02-FPH-254-A3, header_female_3pin:SAMESKY_SSK02-FPH-254-A3, F.Cu at (229.0, 91.8)
- added R15: 0, Resistor_SMD:R_0603_1608Metric, F.Cu at (210.3, 80.7)
- added R16: 0, Resistor_SMD:R_0603_1608Metric, F.Cu at (205.1, 80.0)
- added U10: PCM5102APW, Package_SO:Texas_PW0020A_TSSOP-20_4.4x6.5mm_P0.65mm, F.Cu at (188.2, 104.8)
- C10, C11, C6, C7: footprint Capacitor_SMD:CP_Elec_5x4.5 -> Capacitor_SMD:C_0603_1608Metric
- C8, C9: value 1mF -> 1uF; footprint Capacitor_SMD:CP_Elec_10x10.5 -> Capacitor_SMD:C_0603_1608Metric
- moved C25 195.9 mm to (239.5, 138.2), turned to 180 degrees
- moved C24 190.8 mm to (226.4, 148.3), turned to 180 degrees
- moved C26 172.5 mm to (227.5, 124.2)
- moved C27 167.7 mm to (227.6, 129.3)
- moved C8 155.3 mm to (235.9, 75.3), turned to 90 degrees
- moved C9 143.7 mm to (221.1, 80.7)
- moved C22 85.1 mm to (178.7, 96.8), turned to 90 degrees
- moved C10 81.3 mm to (196.3, 124.8)
- moved C11 70.2 mm to (237.4, 133.6), turned to 180 degrees
- moved C32 66.6 mm to (211.8, 134.0), turned to 90 degrees
- moved C30 65.6 mm to (192.8, 134.1), turned to 90 degrees
- moved C35 63.0 mm to (207.3, 134.1), turned to 90 degrees
- moved C20 51.4 mm to (195.0, 116.0), turned to -90 degrees
- moved U12 48.7 mm to (209.5, 140.0), turned to 180 degrees
- moved U15 46.4 mm to (181.0, 140.0), turned to 180 degrees
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Connections:
- A1 pad 1: unconnected-(A1-GPIO0-Pad1)_1 -> GPIO0
- A1 pad 10: unconnected-(A1-GPIO7-Pad10) -> GPIO7
- A1 pad 11: unconnected-(A1-GPIO8-Pad11)_1 -> GPIO8
- A1 pad 12: unconnected-(A1-GPIO9-Pad12) -> GPIO9
- A1 pad 2: unconnected-(A1-GPIO1-Pad2)_1 -> GPIO1
- A1 pad 20: unconnected-(A1-GPIO15-Pad20)_1 -> GPIO15
- A1 pad 21: unconnected-(A1-GPIO16-Pad21)_1 -> GPIO16
- A1 pad 22: unconnected-(A1-GPIO17-Pad22)_1 -> GPIO17
- A1 pad 24: unconnected-(A1-GPIO18-Pad24)_1 -> GPIO18
- A1 pad 34: unconnected-(A1-GPIO28_ADC2-Pad34) -> GPIO28
- A1 pad 36: unconnected-(A1-3V3-Pad36) -> Screen_Vcc
- A1 pad 6: unconnected-(A1-GPIO4-Pad6) -> GPIO4
- A1 pad 7: unconnected-(A1-GPIO5-Pad7) -> GPIO5
- A1 pad 9: unconnected-(A1-GPIO6-Pad9)_1 -> GPIO6
- C1 pad 2: Net-(D2-COM) -> /pcm_1808/R-ch IN
- C10 pad 2: +9V -> GND
- C11 pad 1: +9V -> GND
- C11 pad 2: +9V -> -9V
- C12 pad 2: GNDA -> GND
- C13 pad 2: GNDA -> GND
- C15 pad 2: GNDA -> GND
- C16 pad 2: GNDA -> GND
- C17 pad 2: +9V -> GND
- C18 pad 2: +9V -> GND
- C19 pad 2: GNDA -> GND
- C2 pad 2: Net-(D2-COM) -> /pcm_1808/L-ch IN
- C20 pad 2: GNDA -> GND
- C21 pad 2: +9V -> GND
- C22 pad 2: +9V -> GND
- C23 pad 2: GNDA -> GND
- C25 pad 1: +9V -> GND
- C25 pad 2: +9V -> -9V
- C26 pad 2: +9V -> GND
- C27 pad 2: +9V -> GND
- C28 pad 2: +9V -> GND
- C29 pad 2: +9V -> GND
- C3 pad 2: +9V -> GND
- C30 pad 2: +9V -> GND
- C31 pad 2: +9V -> GND
- C32 pad 2: +9V -> GND
- C33 pad 2: +9V -> GND
- C34 pad 2: +9V -> GND
- C35 pad 2: +9V -> GND
- C4 pad 1: GNDA -> GND
- C5 pad 2: +9V -> GND
- C7 pad 2: +9V -> GND
- C9 pad 1: +9V -> GND
- R1 pad 2: +9V -> GND
- R10 pad 1: +9V -> GND
- R2 pad 1: +9V -> GND
- R3 pad 1: +9V -> GND
- R6 pad 2: +9V -> GND
- R7 pad 1: +9V -> GND
- R8 pad 2: +9V -> -9V
- U1 pad 3: +9V -> GND
- U1 pad 5: +9V -> -9V
- U12 pad 2: +9V -> GND
- U13 pad 2: +9V -> GND
- U14 pad 2: +9V -> GND
- U15 pad 2: +9V -> GND
- U5 pad 10: +9V -> GND
- U5 pad 11: +9V -> GND
- U5 pad 12: +9V -> GND
- U5 pad 2: GNDA -> GND
- U5 pad 5: +9V -> GND
- U7 pad 4: (no net) -> -9V
- U7 pad 8: (no net) -> +9V
Routing:
- net +9V: track 8.54 -> 209.9 mm, vias 0 -> 4
- net -9V: track 0.00 -> 120.4 mm
- net +5VA: track 7.96 -> 123.6 mm
- net GNDA: track 49.1 -> 0.00 mm
- net +3.3VA: track 2.96 -> 48.9 mm
- net GND: track 0.00 -> 42.1 mm, vias 0 -> 19
- net +3V3: track 5.07 -> 38.5 mm
- net BCK: track 41.0 -> 69.6 mm, vias 1 -> 4
- net DAC Dout: track 0.17 -> 27.1 mm, vias 0 -> 1
- net Net-(U1-CAP-): track 0.00 -> 14.1 mm
- net Net-(D2-COM): track 30.4 -> 16.6 mm, vias 0 -> 2
- net GPIO9: track 0.00 -> 11.8 mm
- net GPIO16: track 0.00 -> 11.4 mm
- net MCK: track 43.5 -> 54.4 mm, vias 2 -> 0
- net GPIO6: track 0.00 -> 10.9 mm
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- added copper zone on B.Cu, net GND
- added copper zone on F.Cu, net GND
Other:
- board outline added: 100 x 100 mm
- board text removed: "sigout"

Commit message: Adding PCB changes, so Luke's ss stuff don't break my stuff
Parts:
- removed C2: 1uF, Capacitor_SMD:CP_Elec_4x5.7
- removed R14, R15: 0, Resistor_SMD:R_0603_1608Metric
- moved R10 21.2 mm to (220.3, 62.1), turned to -90 degrees
- moved R6 19.4 mm to (222.1, 80.7)
- moved R7 17.7 mm to (212.8, 68.8), turned to 0 degrees
- moved R1 17.0 mm to (246.6, 76.9), turned to -90 degrees
- moved C8 15.1 mm to (225.8, 64.1), turned to 180 degrees
- moved R9 15.0 mm to (223.0, 62.1)
- moved R8 14.9 mm to (217.1, 70.3), turned to 90 degrees
- moved C7 14.0 mm to (225.5, 79.9)
- moved R5 13.2 mm to (230.1, 78.8), turned to 180 degrees
- moved C9 11.5 mm to (214.0, 71.7)
- moved R2 10.5 mm to (243.8, 69.0)
- moved C6 10.2 mm to (244.9, 72.4)
- moved R4 9.76 mm to (238.1, 78.7), turned to 180 degrees
- moved U7 9.63 mm to (223.7, 68.4), turned to 0 degrees
- moved R3 9.45 mm to (242.7, 76.9), turned to 90 degrees
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Connections:
- C1 pad 2: /pcm_1808/R-ch IN -> Net-(D2-COM)
- C9 pad 2: Net-(U8A-+) -> 2IN+
- R7 pad 2: Net-(U8A-+) -> 2IN+
- R8 pad 1: Net-(U8A-+) -> 2IN+
- U5 pad 13: Net-(U5-VINL) -> Net-(U5-VINR)
- U6 pad 4: (no net) -> -9V
- U6 pad 8: (no net) -> +9V
- U7 pad 5: (no net) -> 2IN+
- U7 pad 6: (no net) -> Net-(D2-A)
- U7 pad 7: (no net) -> Net-(D2-A)
Routing:
- net +9V: track 209.9 -> 242.0 mm, vias 4 -> 2
- net -9V: track 120.4 -> 150.7 mm, vias 0 -> 2
- net 2IN+: track 0.00 -> 15.0 mm, vias 0 -> 2
- net Net-(D2-A): track 0.00 -> 8.89 mm
- net Net-(D2-K): track 0.00 -> 8.89 mm
- net Net-(U6A--): track 7.57 -> 15.0 mm
- net Net-(U5-VINL): track 5.76 -> 0.00 mm
- net Net-(U8A-+): track 4.65 -> 0.00 mm
- net Net-(U6A-+): track 6.73 -> 11.2 mm
- net Net-(C2-Pad1): track 3.79 -> 0.00 mm
- net Net-(U7A-+): track 14.9 -> 12.5 mm
- net Net-(U5-VINR): track 7.37 -> 9.48 mm
- net Net-(D2-COM): track 16.6 -> 17.8 mm, vias 2 -> 0
- net /AnalogFE/Guitar_In: track 2.77 -> 3.72 mm
- net +3V3: track 38.5 -> 39.4 mm
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
Commit message: First iteration, need to tweak some things
Parts:
- removed J11: P_Switch, header_female_2pin:SAMESKY_SSK02-FPH-254-A2
- removed U12: MCP1703T-3302E/DB, lin_reg:SOT-223_3MC_MCH
- added C2: 10uF, Capacitor_SMD:C_1206_3216Metric, F.Cu at (238.0, 69.7)
- added C36: .1uF, Capacitor_SMD:C_0402_1005Metric_Pad0.74x0.62mm_HandSolder, F.Cu at (218.0, 67.7)
- added C37: .1uF, Capacitor_SMD:C_0402_1005Metric_Pad0.74x0.62mm_HandSolder, F.Cu at (228.9, 65.7)
- added C38: 10uF, Capacitor_SMD:C_1206_3216Metric, F.Cu at (230.1, 67.4)
- added C39: 10uF, Capacitor_SMD:C_1206_3216Metric, F.Cu at (227.0, 75.8)
- added C40: .1uF, Capacitor_SMD:C_0402_1005Metric_Pad0.74x0.62mm_HandSolder, F.Cu at (228.1, 72.1)
- added D1: 1N5819, 1N45819:1N5819HW-7-F_DIO-M, F.Cu at (248.1, 123.2)
- added J14: powerRailAndBatteryGround, header_fem_pin2:SAMESKY_SSK02-FPH-254-A2, F.Cu at (179.4, 128.7)
- added J16: Barrel3andbarrel2, header_fem_pin2:SAMESKY_SSK02-FPH-254-A2, F.Cu at (180.3, 124.0)
- added J17: Guitar input, header_fem_pin2:SAMESKY_SSK02-FPH-254-A2, F.Cu at (251.1, 73.7)
- added J18: positivePowerInputs, header_fem_pin3:SAMESKY_SSK02-FPH-254-A3, F.Cu at (190.6, 129.2)
- added J19: positivePowerInputs, header_fem_pin3:SAMESKY_SSK02-FPH-254-A3, F.Cu at (187.1, 120.3)
- added R14: 22, Resistor_SMD:R_0402_1005Metric_Pad0.72x0.64mm_HandSolder, F.Cu at (217.6, 95.0)
- added R15: 22, Resistor_SMD:R_0402_1005Metric_Pad0.72x0.64mm_HandSolder, F.Cu at (215.1, 95.3)
- added R17: 22, Resistor_SMD:R_0402_1005Metric_Pad0.72x0.64mm_HandSolder, F.Cu at (212.5, 95.3)
- added R18: 22, Resistor_SMD:R_0402_1005Metric_Pad0.72x0.64mm_HandSolder, F.Cu at (190.4, 98.6)
- added R19: 22, Resistor_SMD:R_0402_1005Metric_Pad0.72x0.64mm_HandSolder, F.Cu at (209.9, 85.6)
- added TP1: TestPoint, TestPoint:TestPoint_Loop_D2.50mm_Drill1.85mm, F.Cu at (248.2, 68.4)
- added TP2: TestPoint, TestPoint:TestPoint_Loop_D2.50mm_Drill1.85mm, F.Cu at (216.4, 81.5)
- added TP3: TestPoint, TestPoint:TestPoint_Loop_D2.50mm_Drill1.85mm, F.Cu at (188.4, 68.5)
- added TP4: TestPoint, TestPoint:TestPoint_Loop_D2.50mm_Drill1.85mm, F.Cu at (236.6, 83.0)
- added TP5: TestPoint, TestPoint:TestPoint_Loop_D2.50mm_Drill1.85mm, F.Cu at (219.5, 91.4)
- added U2: PMEG2005CT_215, powa_protec_dat_diode:SOT_05CT215_NEX-M, F.Cu at (191.1, 125.3)
- C32: value 1uF -> .1uF; footprint Capacitor_SMD:C_0603_1608Metric -> Capacitor_SMD:C_0402_1005Metric_Pad0.74x0.62mm_HandSolder
- C35: value 1uF -> 10uF; footprint Capacitor_SMD:C_0603_1608Metric -> Capacitor_SMD:C_1206_3216Metric
- J1, J7, J8: footprint header_female_2pin:SAMESKY_SSK02-FPH-254-A2 -> header_fem_pin2:SAMESKY_SSK02-FPH-254-A2
- J10: value Battery in -> footswitch3; footprint header_female_2pin:SAMESKY_SSK02-FPH-254-A2 -> header_fem_pin2:SAMESKY_SSK02-FPH-254-A2
- J2, J3, J4, J9: footprint header_female_3pin:SAMESKY_SSK02-FPH-254-A3 -> header_fem_pin3:SAMESKY_SSK02-FPH-254-A3
- J5: value SSK02-FPH-254-A2 -> footswitch1; footprint header_female_2pin:SAMESKY_SSK02-FPH-254-A2 -> header_fem_pin2:SAMESKY_SSK02-FPH-254-A2
- J6: value SSK02-FPH-254-A2 -> footswitch2; footprint header_female_2pin:SAMESKY_SSK02-FPH-254-A2 -> header_fem_pin2:SAMESKY_SSK02-FPH-254-A2
- moved C32 69.1 mm to (236.1, 69.4), turned to -90 degrees
- moved C35 63.7 mm to (217.9, 71.2), turned to -90 degrees
- moved J6 55.6 mm to (201.2, 123.2), turned to 90 degrees
- moved J5 54.3 mm to (197.7, 104.4), turned to 90 degrees
- moved J10 38.1 mm to (232.7, 121.5), turned to 180 degrees
- moved J1 34.1 mm to (250.6, 92.5), turned to 90 degrees
- moved J3 30.6 mm to (225.5, 91.6), turned to 90 degrees
- moved J9 30.0 mm to (225.2, 121.5), turned to 0 degrees
- moved C10 13.1 mm to (184.0, 129.4), turned to 90 degrees
- moved C26 10.7 mm to (217.3, 127.2), turned to 90 degrees
- moved R8 4.36 mm to (212.7, 70.0)
- moved R7 4.36 mm to (208.4, 68.6)
- moved C9 4.36 mm to (209.6, 71.5)
- moved J2 3.45 mm to (229.1, 91.7), turned to -90 degrees
- moved C12 2.20 mm to (189.9, 118.2)
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Connections:
- net 2IN+ renamed Net-(U7B-+)
- net Net-(D2-COM) renamed GuitarIn
- A1 pad 14: MCK -> Net-(A1-GPIO10)
- A1 pad 15: BCK -> Net-(A1-GPIO11)
- A1 pad 16: LRCK -> Net-(A1-GPIO12)
- A1 pad 2: GPIO1 -> unconnected-(A1-GPIO1-Pad2)
- A1 pad 29: unconnected-(A1-GPIO22-Pad29)_1 -> GPIO22
- A1 pad 31: unconnected-(A1-GPIO26_ADC0-Pad31) -> GPIO26
- A1 pad 32: unconnected-(A1-GPIO27_ADC1-Pad32) -> GPIO27
- A1 pad 34: GPIO28 -> unconnected-(A1-GPIO28_ADC2-Pad34)
- A1 pad 39: unconnected-(A1-VSYS-Pad39)_1 -> Net-(A1-VSYS)
- C17 pad 1: +3V3 -> Screen_Vcc
- C22 pad 1: +3V3 -> Screen_Vcc
- C3 pad 1: +3V3 -> Screen_Vcc
- C32 pad 1: +9V -> GND
- C32 pad 2: GND -> -9V
- C35 pad 1: +3.3V -> -9V
- J1 pad 1: GPIO28 -> GPIO0
- J10 pad 1: unconnected-(J10-Pad1) -> GND
- J10 pad 2: +9V -> GPIO27
- J2 pad 1: GPIO8 -> GPIO6
- J2 pad 3: GPIO9 -> GPIO7
- J3 pad 1: GPIO15 -> GPIO8
- J3 pad 3: GPIO16 -> GPIO9
- J5 pad 2: GPIO0 -> GPIO15
- J6 pad 2: GPIO1 -> GPIO16
- J7 pad 1: GPIO5 -> GPIO4
- J7 pad 2: GPIO4 -> GPIO5
- J9 pad 1: GPIO6 -> GPIO22
- J9 pad 3: GPIO7 -> GPIO26
- U10 pad 14: DAC Dout -> Net-(U10-DIN)
- U10 pad 20: +3V3 -> Screen_Vcc
- U5 pad 4: +3V3 -> Screen_Vcc
- U5 pad 9: ADC Din -> Net-(U5-DOUT)
- U6 pad 5: (no net) -> GND
- U6 pad 6: (no net) -> Net-(U6B--)
- U6 pad 7: (no net) -> Net-(U6B--)
Routing:
- net Screen_Vcc: track 3.67 -> 143.3 mm, vias 0 -> 4
- net +5VD: track 1.94 -> 85.4 mm, vias 0 -> 2
- net GND: track 42.1 -> 123.0 mm, vias 24 -> 52
- net +3V3: track 39.4 -> 0.00 mm
- net -9V: track 150.7 -> 184.9 mm, vias 2 -> 4
- net +9V: track 242.0 -> 230.0 mm, vias 2 -> 4
- net /AnalogFE/Guitar_In: track 3.72 -> 13.0 mm
- net GuitarIn: track 17.8 -> 25.1 mm
- net GPIO16: track 11.4 -> 4.71 mm
- net Net-(J18-Pad3): track 0.00 -> 6.38 mm
- net GPIO1: track 5.60 -> 0.00 mm
- net GPIO28: track 4.94 -> 0.00 mm
- net Net-(U2-common_cathode): track 0.00 -> 4.75 mm
- net LRCK: track 41.6 -> 37.2 mm
- net Net-(J14-Pad2): track 0.00 -> 4.40 mm
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Other:
- board size 100 x 100 mm -> 96.1 x 96.7 mm
