File: KiCad/pcm_1808.kicad_sch (KiCad schematic)
At the start: 10 parts, among them U5 PCM1808-Q1_PW_14

Commit message: PCB ex
Connections:
- net GNDA is gone; now on net GND: C36.2, C37.2, C4.1, U5.2 (AGND)
Changed lines of the file:
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@@
+	)
+	(junction
+		(at 74.93 76.2)
+		(diameter 0)
+		(color 0 0 0 0)
 	)
 	(junction
@@
 		(color 0 0 0 0)
 	)
+	(junction
+		(at 90.17 96.52)
+		(diameter 0)
+		(color 0 0 0 0)
+	)
 	(wire
 		(pts
@@
 	(wire
 		(pts
+			(xy 74.93 76.2) (xy 74.93 96.52)
+		)
+		(stroke
+			(width 0)
+			(type default)
+		)
+	)
+	(wire
+		(pts
 			(xy 196.85 80.01) (xy 196.85 74.93)
 		)
@@
 	(wire
 		(pts
+			(xy 74.93 96.52) (xy 90.17 96.52)
+		)
+		(stroke
+			(width 0)
+			(type default)
+		)
+	)
+	(wire
+		(pts
 			(xy 101.6 88.9) (xy 101.6 82.55)
 		)
@@
 	(wire
 		(pts
-			(xy 71.12 76.2) (xy 83.82 76.2)
+			(xy 71.12 76.2) (xy 74.93 76.2)
 		)
 		(stroke
@@
 	(wire
 		(pts
-			(xy 90.17 85.09) (xy 90.17 100.33)
+			(xy 90.17 85.09) (xy 90.17 96.52)
 		)
 		(stroke
@@
 		)
 		(stroke
+			(width 0)
+			(type default)
+		)
+	)
+	(wire
+		(pts
+			(xy 74.93 76.2) (xy 83.82 76.2)
+		)
+		(stroke
+			(width 0)
+			(type default)
+		)
+	)
+	(wire
+		(pts
+			(xy 90.17 96.52) (xy 90.17 100.33)
+		)
+		(stroke
