File: KiCad/pcm_1808.kicad_sch (KiCad schematic)
At the start: 8 parts, among them U5 PCM1808-Q1_PW_14

Commit message: Changes to the BoM
Parts:
- C1: Part_Number (none) -> 865060640001
- C3, C4: Part_Number (none) -> C0603C104K5RACTU
- C5: Part_Number (none) -> UWT1H100MCL1GB
- R19: Part_Number (none) -> CRCW040222R0FKED
- U5: Part_Number (none) -> PCM1808PWR
Changed lines of the file:
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@@
 			)
 		)
-		(property "Datasheet" ""
+		(property "Datasheet" "https://www.digikey.com/en/products/detail/kemet/C0603C104K5RACTU/1465594"
 			(at 83.82 78.74 0)
 			(hide yes)
@@
 		)
 		(property "Description" "Unpolarized capacitor, small symbol"
+			(at 83.82 78.74 0)
+			(hide yes)
+			(show_name no)
+			(do_not_autoplace no)
+			(effects
+				(font
+					(size 1.27 1.27)
+				)
+			)
+		)
+		(property "Part_Number" "C0603C104K5RACTU"
 			(at 83.82 78.74 0)
 			(hide yes)
@@
 			)
 		)
-		(property "Datasheet" ""
+		(property "Datasheet" "https://industrial.panasonic.com/cdbs/www-data/pdf/RDA0000/AOA0000C304.pdf"
 			(at 196.85 82.55 0)
 			(hide yes)
@@
 		)
 		(property "Description" "Resistor, US symbol"
+			(at 196.85 82.55 0)
+			(hide yes)
+			(show_name no)
+			(do_not_autoplace no)
+			(effects
+				(font
+					(size 1.27 1.27)
+				)
+			)
+		)
+		(property "Part_Number" ""
 			(at 196.85 82.55 0)
 			(hide yes)
@@
 			)
 		)
-		(property "Datasheet" ""
+		(property "Datasheet" "https://www.digikey.com/en/products/detail/w%C3%BCrth-elektronik/865060640001/5728136?s=N4IgTCBcDaIBwDYCsAGBaAsLsEYQF0BfIA"
 			(at 226.06 74.93 0)
 			(hide yes)
@@
 		)
 		(property "Description" "Polarized capacitor, small US symbol"
+			(at 226.06 74.93 0)
+			(hide yes)
+			(show_name no)
+			(do_not_autoplace no)
+			(effects
+				(font
+					(size 1.27 1.27)
+				)
+			)
+		)
+		(property "Part_Number" "865060640001"
 			(at 226.06 74.93 0)
 			(hide yes)
@@
 			)
 		)
-		(property "Datasheet" ""
+		(property "Datasheet" "https://www.digikey.com/en/products/detail/kemet/C0603C104K5RACTU/1465594"
 			(at 101.6 91.44 0)
 			(hide yes)
@@
 		)
 		(property "Description" "Unpolarized capacitor, small symbol"
+			(at 101.6 91.44 0)
+			(hide yes)
+			(show_name no)
+			(do_not_autoplace no)
+			(effects
+				(font
+					(size 1.27 1.27)
+				)
+			)
+		)
+		(property "Part_Number" "C0603C104K5RACTU"
 			(at 101.6 91.44 0)
 			(hide yes)
@@
 			)
 		)
-		(property "Datasheet" ""
+		(property "Datasheet" "https://industrial.panasonic.com/cdbs/www-data/pdf/RDA0000/AOA0000C304.pdf"
 			(at 201.93 74.93 0)
 			(hide yes)
@@
 		(property "Description" "Resistor, US symbol"
 			(at 201.93 74.93 0)
+			(hide yes)
+			(show_name no)
+			(do_not_autoplace no)
+			(effects
+				(font
+					(size 1.27 1.27)
+				)
+			)
+		)
+		(property "Part_Number" ""
+			(at 201.93 74.93 90)
 			(hide yes)
 			(show_name no)
@@
 			)
 		)
+		(property "Part_Number" "PCM1808PWR"
+			(at 118.11 74.93 0)
+			(hide yes)
+			(show_name no)
+			(do_not_autoplace no)
+			(effects
+				(font
+					(size 1.27 1.27)
+				)
+			)
+		)
 		(pin "2"
 		)
@@
 			)
 		)
-		(property "Datasheet" ""
+		(property "Datasheet" "https://www.nichicon.co.jp/english/series_items/catalog_pdf/e-uwt.pdf"
 			(at 114.3 74.93 0)
 			(hide yes)
@@
 		(property "Description" "Polarized capacitor, small US symbol"
 			(at 114.3 74.93 0)
+			(hide yes)
+			(show_name no)
+			(do_not_autoplace no)
+			(effects
+				(font
+					(size 1.27 1.27)
+				)
+			)
+		)
+		(property "Part_Number" "UWT1H100MCL1GB"
+			(at 114.3 74.93 90)
 			(hide yes)
 			(show_name no)
@@
 			)
 		)
-		(property "Datasheet" ""
+		(property "Datasheet" "https://www.digikey.com/en/products/detail/vishay-dale/CRCW040222R0FKED/1177815"
 			(at 186.69 91.44 0)
 			(hide yes)
@@
 			(at 186.69 91.44 0)
 			(hide yes)
+			(show_name no)
+			(do_not_autoplace no)
+			(effects
+				(font
+					(size 1.27 1.27)
+				)
+			)
+		)
+		(property "Part_Number" "CRCW040222R0FKED"
+			(at 186.69 91.44 0)
+			(hide yes)
