File: KiCad/rpi_and_peripherals.kicad_sch (KiCad schematic)
At the start: 5 parts, among them U2 RP2350A, U3 PCM5102A, U4 PCM1808-Q1_PW_14

Commit message: Testing repository on laptop
Changed lines of the file:
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@@
 		)
 	)
-	(text_box "TODO:\n1. Investigate settings on the DAC & ADC to verify they align with the schematic.\n2. Investigate the CAPM, CAPP, & the LDOO signals on the DAC.\n3. Look into the backend on the board currently being used by the system, is there one?\n4. Fill out schematics on the FE & BE. "
+	(text_box "TODO:\n1. Investigate settings on the DAC & ADC to verify they align with the schematic.\n2. Investigate the CAPM, CAPP, & the LDOO signals on the DAC.\n3. Look into the backend on the board currently being used by the system, is there one?\n4. Fill out schematics on the FE & BE. \n5. Need to fix RP2350A, find footprint of the devkit rather than the processor. "
 		(exclude_from_sim no)
 		(at 163.83 100.33 0)
-		(size 67.31 16.51)
+		(size 67.31 22.86)
 		(margins 0.9525 0.9525 0.9525 0.9525)
 		(stroke

Commit message: First PCB layout iteration, custom footprint for Pico
Parts:
- removed U2: RP2350A, Package_DFN_QFN:QFN-60-1EP_7x7mm_P0.4mm_EP3.4x3.4mm, symbol MCU_RaspberryPi:RP2350A
- added U2: (no value), rpi_foot:rpi_dev_foot, symbol PCM1808:Pico_Dev_Board
- AnalogBE1: renamed from AnalogBE; now left out of the parts list
- AnalogFE1: renamed from AnalogFE; now left out of the parts list
Connections:
- net +3V3: now also U3.1 (CPVDD), U3.20 (DVDD), U3.8 (AVDD)
- net ADC Din: now also U2.19 (GPIO14)
- net BCK: now also U2.15 (GPIO11)
- net DAC Dout: now also U2.17 (GPIO13)
- net DEBUG_LED1: now also U2.31 (GPIO19)
- net DEBUG_LED2: now also U2.32 (GPIO20)
- net DEBUG_LED3: now also U2.33 (GPIO21)
- net GND: now also U2.38 (GND), U2.8 (GND)
- net LRCK: now also U2.16 (GPIO12)
- net MCK: now also U2.14 (GPIO10)
- net PICO_DEBUG: now also U2.36 (3V3(OUT))
- net -3V3: now reaches U3.5 (VNEG)
- net G_Lout: now reaches AnalogFE1. (Rout), U4.13 (VINL)
- net G_Rout: now reaches AnalogFE1. (Rout), U4.14 (VINR)

Commit message: Filled out FE schematic block
Connections:
- net +9V: now reaches AnalogFE1.3 (V++)
- net +9V: now also AnalogBE1.3 (V++)
- net -9V: now reaches AnalogFE1.4 (V--)
- net -9V: now also AnalogBE1.4 (V--)
- net PICO_DEBUG: no longer names the net of U2.36 (3V3(OUT))
Changed lines of the file:
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@@
 		)
 	)
-	(text_box "TODO:\n1. Investigate settings on the DAC & ADC to verify they align with the schematic.\n2. Investigate the CAPM, CAPP, & the LDOO signals on the DAC.\n3. Look into the backend on the board currently being used by the system, is there one?\n4. Fill out schematics on the FE & BE. \n5. Need to fix RP2350A, find footprint of the devkit rather than the processor. "
+	(text_box "TODO:\n1. Investigate settings on the DAC & ADC to verify they align with the schematic.\n2. Investigate the CAPM, CAPP, & the LDOO signals on the DAC.\n3. Look into the backend on the board currently being used by the system, is there one?\n4. Fill out schematics on BE and verify the FE schem with Luke.\n5. Need to fix RP2350A, find footprint of the devkit rather than the processor. "
 		(exclude_from_sim no)
 		(at 163.83 100.33 0)
-		(size 67.31 22.86)
+		(size 67.31 20.3053)
 		(margins 0.9525 0.9525 0.9525 0.9525)
 		(stroke
@@
 	)
 	(junction
+		(at 107.95 105.41)
+		(diameter 0)
+		(color 0 0 0 0)
+	)
+	(junction
 		(at 146.05 85.09)
 		(diameter 0)
@@
 	)
 	(junction
-		(at 106.68 105.41)
-		(diameter 0)
-		(color 0 0 0 0)
-	)
-	(junction
 		(at 212.09 85.09)
 		(diameter 0)
@@
 	(wire
 		(pts
-			(xy 106.68 105.41) (xy 107.95 105.41)
-		)
-		(stroke
-			(width 0)
-			(type default)
-		)
-	)
-	(wire
-		(pts
 			(xy 106.68 92.71) (xy 214.63 92.71)
 		)
@@
 	(wire
 		(pts
+			(xy 107.95 105.41) (xy 106.68 105.41)
+		)
+		(stroke
+			(width 0)
+			(type default)
+		)
+	)
+	(wire
+		(pts
 			(xy 204.47 34.29) (xy 217.17 34.29)
 		)
@@
 		(pts
 			(xy 151.13 87.63) (xy 106.68 87.63)
-		)
-		(stroke
-			(width 0)
-			(type default)
-		)
-	)
-	(wire
-		(pts
-			(xy 106.68 102.87) (xy 110.49 102.87)
 		)
 		(stroke
@@
 					(size 1.27 1.27)
 				)
+			)
+		)
+	)
+	(global_label "+9V"
+		(shape input)
+		(at 185.42 38.1 180)
+		(fields_autoplaced yes)
+		(effects
+			(font
+				(size 1.27 1.27)
+			)
+			(justify right)
+		)
+		(property "Intersheetrefs" "${INTERSHEET_REFS}"
+			(at 178.5643 38.1 0)
+			(hide yes)
+			(show_name no)
+			(do_not_autoplace no)
+			(effects
+				(font
+					(size 1.27 1.27)
+				)
+				(justify right)
 			)
 		)
@@
 		)
 	)
-	(global_label "PICO_DEBUG"
+	(global_label "+9V"
 		(shape input)
-		(at 110.49 102.87 0)
+		(at 151.13 147.32 180)
 		(fields_autoplaced yes)
 		(effects
@@
 				(size 1.27 1.27)
 			)
-			(justify left)
+			(justify right)
 		)
 		(property "Intersheetrefs" "${INTERSHEET_REFS}"
-			(at 125.2076 102.87 0)
-			(hide yes)
-			(show_name no)
-			(do_not_autoplace no)
-			(effects
-				(font
-					(size 1.27 1.27)
-				)
-				(justify left)
+			(at 144.2743 147.32 0)
+			(hide yes)
+			(show_name no)
+			(do_not_autoplace no)
+			(effects
+				(font
+					(size 1.27 1.27)
+				)
+				(justify right)
+			)
+		)
+	)
+	(global_label "-9V"
+		(shape input)
+		(at 151.13 149.86 180)
+		(fields_autoplaced yes)
+		(effects
+			(font
+				(size 1.27 1.27)
+			)
+			(justify right)
+		)
+		(property "Intersheetrefs" "${INTERSHEET_REFS}"
+			(at 144.2743 149.86 0)
+			(hide yes)
+			(show_name no)
+			(do_not_autoplace no)
+			(effects
+				(font
+					(size 1.27 1.27)
+				)
+				(justify right)
 			)
 		)
@@
 		(property "Intersheetrefs" "${INTERSHEET_REFS}"
 			(at 205.1135 48.26 0)
+			(hide yes)
+			(show_name no)
+			(do_not_autoplace no)
+			(effects
+				(font
+					(size 1.27 1.27)
+				)
+				(justify right)
+			)
+		)
+	)
+	(global_label "-9V"
+		(shape input)
+		(at 185.42 40.64 180)
+		(fields_autoplaced yes)
+		(effects
+			(font
+				(size 1.27 1.27)
+			)
+			(justify right)
+		)
+		(property "Intersheetrefs" "${INTERSHEET_REFS}"
+			(at 178.5643 40.64 0)
 			(hide yes)
 			(show_name no)
@@
 	(symbol
 		(lib_id "power:GND")
-		(at 106.68 105.41 0)
+		(at 107.95 105.41 0)
 		(unit 1)
 		(body_style 1)
@@
 		(fields_autoplaced yes)
 		(property "Reference" "#PWR015"
-			(at 106.68 111.76 0)
+			(at 107.95 111.76 0)
 			(hide yes)
 			(show_name no)
@@
 		)
 		(property "Value" "GND"
-			(at 106.68 110.49 0)
+			(at 107.95 110.49 0)
 			(show_name no)
 			(do_not_autoplace no)
@@
 		)
 		(property "Footprint" ""
-			(at 106.68 105.41 0)
+			(at 107.95 105.41 0)
 			(hide yes)
 			(show_name no)
@@
 		)
 		(property "Datasheet" ""
-			(at 106.68 105.41 0)
+			(at 107.95 105.41 0)
 			(hide yes)
 			(show_name no)
@@
 		)
 		(property "Description" "Power symbol creates a global label with name \"GND\" , ground"
-			(at 106.68 105.41 0)
-			(hide yes)
-			(show_name no)
+			(at 107.95 105.41 0)
+			(hide yes)
+			(show_name no)

Commit message: Changed footprints, added powersystem
Parts:
- removed U3: PCM5102A, Package_SO:TSSOP-20_4.4x6.5mm_P0.65mm, symbol Audio:PCM5102A
- added U3: LT1054, charge_pump:SOIC127P1030X265-16N, symbol Regulator_SwitchedCapacitor:LT1054
- added U9: PCM5102APW, Package_SO:Texas_PW0020A_TSSOP-20_4.4x6.5mm_P0.65mm, symbol DAC:PCM5102APW
- AnalogBE1, AnalogFE1: now in the parts list
- U2, U4: now left out of the parts list
Connections:
- net +3V3: now also U9.1 (CPVDD), U9.20 (DVDD), U9.8 (AVDD)
- net +9V: now also U3.8 (V+)
- net -3V3: now also U9.5 (VNEG)
- net -9V: now also U3.5 (-VOUT)
- net BCK: now also U9.13 (BCK)
- net DAC Dout: now also U9.14 (DIN)
- net GND: now also U3.3 (GND), U9.10 (DEMP), U9.11 (FLT), U9.16 (FMT), U9.17 (XSMT), U9.19 (DGND), U9.3 (CPGND), U9.9 (AGND)
- net LRCK: now also U9.15 (LRCK)
- net MCK: now also U9.12 (SCK)
- net at AnalogBE1.1 (DAC_L): now also U9.6 (OUTL)
- net at AnalogBE1.2 (DAC_R): now also U9.7 (OUTR)
- new net: U3.2 (CAP+), U3.4 (CAP-)
Other:
- added sheet PowerSystem (PowerSystem.kicad_sch)
- moved on the sheet: AnalogBE1

Commit message: Updates for 10_18_26
Other:
- moved on the sheet: AnalogBE1, U3

Commit message: Pushing PCB, and controls schem
Parts:
- removed U2: (no value), rpi_foot:rpi_dev_foot, symbol PCM1808:Pico_Dev_Board
- removed U3: LT1054, charge_pump:SOIC127P1030X265-16N, symbol Regulator_SwitchedCapacitor:LT1054
- added A1: RaspberryPi_Pico, Module:RaspberryPi_Pico_Common_Unspecified, symbol MCU_Module:RaspberryPi_Pico
Connections:
- net +3V3: no longer U9.1 (CPVDD), U9.8 (AVDD)
- net ADC Din: now also A1.19 (GPIO14)
- net BCK: now also A1.15 (GPIO11)
- net DAC Dout: now also A1.17 (GPIO13)
- net LRCK: now also A1.16 (GPIO12)
- net MCK: now also A1.14 (GPIO10)
- net +5V renamed +5VA
- net -3V3: no longer names the net of U9.5 (VNEG)
- new net: A1.13 (GND), A1.18 (GND), A1.23 (GND), A1.28 (GND), A1.3 (GND), A1.38 (GND), A1.8 (GND)
- new net +3.3VA: U9.1 (CPVDD), U9.8 (AVDD)
- no-connect marks 0 -> 31
Other:
- added sheet Control (control.kicad_sch)
- moved on the sheet: AnalogBE1

Commit message: Luke's commit
Other:
- note added: "1. need guitar input (and footprint) 2. need usb-c connector (and footprint) 3. need footprints for the control system (?) 4. need to add battery switch (and footprint) 5. investigate component choices, ie ratings 6. input filter on adc has two cpacitors, change to 0 ohm resistors with DNI values"
Changed lines of the file:
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@@
 		(company "ECE-494-006")
+	)
+	(text "1. need guitar input (and footprint)\n2. need usb-c connector (and footprint)\n3. need footprints for the control system (?)\n4. need to add battery switch (and footprint)\n5. investigate component choices, ie ratings\n6.  input filter on adc has two cpacitors, change to 0 ohm resistors with DNI values"
+		(exclude_from_sim no)
+		(at 202.184 -18.034 0)
+		(effects
+			(font
+				(size 1.27 1.27)
+			)
+		)
 	)
 	(text_box "Raspberry Pi Pico 2 Dev Board\n"

Commit message: Best one yet
Parts:
- removed AnalogBE1: (no value), symbol PCM1808:Analog_BE
- removed AnalogFE1: (no value), symbol PCM1808:Analoge_FE
- removed U4: PCM1808-Q1_PW_14, PW14_TEX, symbol PCM1808:PCM1808-Q1_PW_14
- removed U9: PCM5102APW, Package_SO:Texas_PW0020A_TSSOP-20_4.4x6.5mm_P0.65mm, symbol DAC:PCM5102APW
Connections:
- net GPIO0: now reaches A1.1 (GPIO0)
- net GPIO7: now reaches A1.10 (GPIO7)
- net GPIO8: now reaches A1.11 (GPIO8)
- net GPIO9: now reaches A1.12 (GPIO9)
- net GPIO1: now reaches A1.2 (GPIO1)
- net GPIO15: now reaches A1.20 (GPIO15)
- net GPIO16: now reaches A1.21 (GPIO16)
- net GPIO17: now reaches A1.22 (GPIO17)
- net GPIO18: now reaches A1.24 (GPIO18)
- net GPIO28: now reaches A1.34 (GPIO28_ADC2)
- net Screen_Vcc: now reaches A1.36 (3V3)
- net GPIO4: now reaches A1.6 (GPIO4)
- net GPIO5: now reaches A1.7 (GPIO5)
- net GPIO6: now reaches A1.9 (GPIO6)
- no-connect marks 31 -> 15
Other:
- moved on the sheet: A1
