File: KiCad/control.kicad_sch (KiCad schematic)
At the start: 7 parts, among them SW1 Encoder 1, SW2 Encoder 2, SW3 Encoder 3, SW4 Encoder 4, SW5 SW_Push, SW6 SW_Push, U11 ER_OLEDM0.91_1x-I2C

Commit message: Best one yet
Parts:
- added J1, J5, J6, J7, J8: SSK02-FPH-254-A2, SSK02-FPH-254-A2:SAMESKY_SSK02-FPH-254-A2, symbol female_headers_2pin:SSK02-FPH-254-A2
- added J2, J3, J4, J9: SSK02-FPH-254-A3, SSK02-FPH-254-A3:SAMESKY_SSK02-FPH-254-A3, symbol female_headers_3pin:SSK02-FPH-254-A3
Connections:
- net GND: now also J1.2, J2.2, J3.2, J4.2, J5.1, J6.1, J8.2, J9.2
- net GPIO0: now also J5.2
- net GPIO1: now also J6.2
- net GPIO15: now also J3.1
- net GPIO16: now also J3.3
- net GPIO17: now also J4.1
- net GPIO18: now also J4.3
- net GPIO28: now also J1.1
- net GPIO4: now also J7.2
- net GPIO5: now also J7.1
- net GPIO6: now also J9.1
- net GPIO7: now also J9.3
- net GPIO8: now also J2.1
- net GPIO9: now also J2.3
- net Screen_Vcc: now reaches U11.2 (VCC)
- net Screen_Vcc: now also J8.1
Other:
- moved on the sheet: SW1, SW2, SW3, SW4, SW5, SW6, U11

Commit message: A bunch of schematic changes
Parts:
- added J10: footswitch3, SSK02-FPH-254-A2:SAMESKY_SSK02-FPH-254-A2, symbol female_headers_2pin:SSK02-FPH-254-A2
- added SW7: SW_Push, symbol Switch:SW_Push
- J5: value SSK02-FPH-254-A2 -> footswitch1
- J6: value SSK02-FPH-254-A2 -> footswitch2
Connections:
- net GPIO1 is gone; now on net GPIO16: J6.2, SW6.2
- net GPIO28 is gone; now on net GPIO0: J1.1, SW1.S1
- net GND: now also J10.1, SW7.1
- net GPIO0: no longer J5.2, SW5.2
- net GPIO15: now also J5.2, SW5.2; no longer J3.1, SW3.A
- net GPIO16: no longer J3.3, SW3.B
- net GPIO4: now also J7.1, U11.4 (SDA); no longer J7.2, U11.3 (SCL)
- net GPIO5: now also J7.2, U11.3 (SCL); no longer J7.1, U11.4 (SDA)
- net GPIO6: now also J2.1, SW2.A; no longer J9.1, SW1.A
- net GPIO7: now also J2.3, SW2.B; no longer J9.3, SW1.B
- net GPIO8: now also J3.1, SW3.A; no longer J2.1, SW2.A
- net GPIO9: now also J3.3, SW3.B; no longer J2.3, SW2.B
- new net GPIO22: J9.1, SW1.A
- new net GPIO26: J9.3, SW1.B
- new net GPIO27: J10.2, SW7.2

Commit message: First iteration, need to tweak some things
Parts:
- J1, J10, J5, J6, J7, J8: footprint SSK02-FPH-254-A2:SAMESKY_SSK02-FPH-254-A2 -> header_fem_pin2:SAMESKY_SSK02-FPH-254-A2
- J2, J3, J4, J9: footprint SSK02-FPH-254-A3:SAMESKY_SSK02-FPH-254-A3 -> header_fem_pin3:SAMESKY_SSK02-FPH-254-A3
Changed lines of the file:
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@@
 			)
 		)
-		(property "Footprint" "SSK02-FPH-254-A2:SAMESKY_SSK02-FPH-254-A2"
+		(property "Footprint" "header_fem_pin2:SAMESKY_SSK02-FPH-254-A2"
 			(at 260.35 83.82 0)
 			(hide yes)
@@
 			)
 		)
-		(property "Footprint" "SSK02-FPH-254-A2:SAMESKY_SSK02-FPH-254-A2"
+		(property "Footprint" "header_fem_pin2:SAMESKY_SSK02-FPH-254-A2"
 			(at 168.91 60.96 0)
 			(hide yes)
@@
 			)
 		)
-		(property "Footprint" "SSK02-FPH-254-A2:SAMESKY_SSK02-FPH-254-A2"
+		(property "Footprint" "header_fem_pin2:SAMESKY_SSK02-FPH-254-A2"
 			(at 146.05 142.24 0)
 			(hide yes)
@@
 			(project "rpi_and_peripherals"
 				(path "/149bebb8-d22c-435a-adf0-1313d3be5660/25a4df0c-f5c6-44f8-9b53-373c76b27ec3"
+					(reference "J10")
+					(unit 1)
+				)
+			)
+			(project "KiCad"
+				(path "/24850b4e-1ce6-41a1-b1f6-c45749a7c3af/25a4df0c-f5c6-44f8-9b53-373c76b27ec3"
 					(reference "J10")
 					(unit 1)
@@
 			)
 		)
-		(property "Footprint" "SSK02-FPH-254-A2:SAMESKY_SSK02-FPH-254-A2"
+		(property "Footprint" "header_fem_pin2:SAMESKY_SSK02-FPH-254-A2"
 			(at 168.91 100.33 0)
 			(hide yes)
@@
 		(exclude_from_sim no)
 		(in_bom yes)
-		(on_board yes)
+		(on_board no)
 		(in_pos_files yes)
 		(dnp no)
@@
 		(exclude_from_sim no)
 		(in_bom yes)
-		(on_board yes)
+		(on_board no)
 		(in_pos_files yes)
 		(dnp no)
@@
 			)
 		)
-		(property "Footprint" "SSK02-FPH-254-A2:SAMESKY_SSK02-FPH-254-A2"
+		(property "Footprint" "header_fem_pin2:SAMESKY_SSK02-FPH-254-A2"
 			(at 241.3 41.91 0)
 			(hide yes)
@@
 		(exclude_from_sim no)
 		(in_bom yes)
-		(on_board yes)
+		(on_board no)
 		(in_pos_files yes)
 		(dnp no)
@@
 			(project "rpi_and_peripherals"
 				(path "/149bebb8-d22c-435a-adf0-1313d3be5660/25a4df0c-f5c6-44f8-9b53-373c76b27ec3"
+					(reference "SW7")
+					(unit 1)
+				)
+			)
+			(project "KiCad"
+				(path "/24850b4e-1ce6-41a1-b1f6-c45749a7c3af/25a4df0c-f5c6-44f8-9b53-373c76b27ec3"
 					(reference "SW7")
 					(unit 1)
@@
 		(exclude_from_sim no)
 		(in_bom yes)
-		(on_board yes)
+		(on_board no)
 		(in_pos_files yes)
 		(dnp no)
@@
 			)
 		)
-		(property "Footprint" "SSK02-FPH-254-A2:SAMESKY_SSK02-FPH-254-A2"
+		(property "Footprint" "header_fem_pin2:SAMESKY_SSK02-FPH-254-A2"
 			(at 124.46 58.42 0)
 			(hide yes)
@@
 			)
 		)
-		(property "Footprint" "SSK02-FPH-254-A3:SAMESKY_SSK02-FPH-254-A3"
+		(property "Footprint" "header_fem_pin3:SAMESKY_SSK02-FPH-254-A3"
 			(at 78.74 78.74 0)
 			(hide yes)
@@
 			)
 		)
-		(property "Footprint" "SSK02-FPH-254-A3:SAMESKY_SSK02-FPH-254-A3"
+		(property "Footprint" "header_fem_pin3:SAMESKY_SSK02-FPH-254-A3"
 			(at 78.74 113.03 0)
 			(hide yes)
@@
 		(exclude_from_sim no)
 		(in_bom yes)
-		(on_board yes)
+		(on_board no)
 		(in_pos_files yes)
 		(dnp no)
@@
 				)
 			)
+			(project "KiCad"
+				(path "/24850b4e-1ce6-41a1-b1f6-c45749a7c3af/25a4df0c-f5c6-44f8-9b53-373c76b27ec3"
+					(reference "#PWR042")
+					(unit 1)
+				)
+			)
 		)
 	)
@@
 			)
 		)
-		(property "Footprint" "SSK02-FPH-254-A3:SAMESKY_SSK02-FPH-254-A3"
+		(property "Footprint" "header_fem_pin3:SAMESKY_SSK02-FPH-254-A3"
 			(at 78.74 39.37 0)
 			(hide yes)
@@
 		(exclude_from_sim no)
 		(in_bom yes)
-		(on_board yes)
+		(on_board no)
 		(in_pos_files yes)
 		(dnp no)
@@
 			)
 		)
-		(property "Footprint" "SSK02-FPH-254-A3:SAMESKY_SSK02-FPH-254-A3"
+		(property "Footprint" "header_fem_pin3:SAMESKY_SSK02-FPH-254-A3"
 			(at 78.74 144.78 0)
 			(hide yes)
@@
 		(exclude_from_sim no)
 		(in_bom yes)
-		(on_board yes)
+		(on_board no)
 		(in_pos_files yes)
 		(dnp no)
@@
 		(exclude_from_sim no)
 		(in_bom yes)
-		(on_board yes)
+		(on_board no)
 		(in_pos_files yes)
 		(dnp no)

Commit message: Changes to the BoM
Parts:
- J1, J10, J5, J6, J7, J8: Part_Number (none) -> SSK02-FPH-254-A2
- J2, J3, J4, J9: Part_Number (none) -> SSK02-FPH-254-A3
Changed lines of the file:
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@@
 			)
 		)
-		(property "Datasheet" ""
+		(property "Datasheet" "https://www.digikey.com/en/products/detail/same-sky-formerly-cui-devices/SSK02-FPH-254-A2/28772215"
 			(at 260.35 83.82 0)
 			(hide yes)
@@
 				)
 				(justify bottom)
+			)
+		)
+		(property "Part_Number" "SSK02-FPH-254-A2"
+			(at 260.35 83.82 0)
+			(hide yes)
+			(show_name no)
+			(do_not_autoplace no)
+			(effects
+				(font
+					(size 1.27 1.27)
+				)
 			)
 		)
@@
 			)
 		)
-		(property "Datasheet" ""
+		(property "Datasheet" "https://www.digikey.com/en/products/detail/same-sky-formerly-cui-devices/SSK02-FPH-254-A2/28772215"
 			(at 168.91 60.96 0)
 			(hide yes)
@@
 				)
 				(justify bottom)
+			)
+		)
+		(property "Part_Number" "SSK02-FPH-254-A2"
+			(at 168.91 60.96 90)
+			(hide yes)
+			(show_name no)
+			(do_not_autoplace no)
+			(effects
+				(font
+					(size 1.27 1.27)
+				)
 			)
 		)
@@
 			)
 		)
-		(property "Datasheet" ""
+		(property "Datasheet" "https://www.digikey.com/en/products/detail/same-sky-formerly-cui-devices/SSK02-FPH-254-A2/28772215"
 			(at 146.05 142.24 0)
 			(hide yes)
@@
 				)
 				(justify bottom)
+			)
+		)
+		(property "Part_Number" "SSK02-FPH-254-A2"
+			(at 146.05 142.24 90)
+			(hide yes)
+			(show_name no)
+			(do_not_autoplace no)
+			(effects
+				(font
+					(size 1.27 1.27)
+				)
 			)
 		)
@@
 			)
 		)
-		(property "Datasheet" ""
+		(property "Datasheet" "https://www.digikey.com/en/products/detail/same-sky-formerly-cui-devices/SSK02-FPH-254-A2/28772215"
 			(at 168.91 100.33 0)
 			(hide yes)
@@
 				)
 				(justify bottom)
+			)
+		)
+		(property "Part_Number" "SSK02-FPH-254-A2"
+			(at 168.91 100.33 90)
+			(hide yes)
+			(show_name no)
+			(do_not_autoplace no)
+			(effects
+				(font
+					(size 1.27 1.27)
+				)
 			)
 		)
@@
 			)
 		)
+		(property "Part_Number" ""
+			(at 99.06 97.79 0)
+			(hide yes)
+			(show_name no)
+			(do_not_autoplace no)
+			(effects
+				(font
+					(size 1.27 1.27)
+				)
+			)
+		)
 		(pin "S1"
 		)
@@
 			)
 		)
+		(property "Part_Number" ""
+			(at 96.52 165.1 0)
+			(hide yes)
+			(show_name no)
+			(do_not_autoplace no)
+			(effects
+				(font
+					(size 1.27 1.27)
+				)
+			)
+		)
 		(pin "S1"
 		)
@@
 			)
 		)
-		(property "Datasheet" ""
+		(property "Datasheet" "https://www.digikey.com/en/products/detail/same-sky-formerly-cui-devices/SSK02-FPH-254-A2/28772215"
 			(at 241.3 41.91 0)
 			(hide yes)
@@
 				)
 				(justify bottom)
+			)
+		)
+		(property "Part_Number" "SSK02-FPH-254-A2"
+			(at 241.3 41.91 90)
+			(hide yes)
+			(show_name no)
+			(do_not_autoplace no)
+			(effects
+				(font
+					(size 1.27 1.27)
+				)
 			)
 		)
@@
 			)
 		)
+		(property "Part_Number" ""
+			(at 147.32 168.91 0)
+			(hide yes)
+			(show_name no)
+			(do_not_autoplace no)
+			(effects
+				(font
+					(size 1.27 1.27)
+				)
+			)
+		)
 		(pin "1"
 		)
@@
 			)
 		)
+		(property "Part_Number" ""
+			(at 242.57 66.04 90)
+			(hide yes)
+			(show_name no)
+			(do_not_autoplace no)
+			(effects
+				(font
+					(size 1.27 1.27)
+				)
+			)
+		)
 		(pin "1"
 		)
@@
 			)
 		)
-		(property "Datasheet" ""
+		(property "Datasheet" "https://www.digikey.com/en/products/detail/same-sky-formerly-cui-devices/SSK02-FPH-254-A2/28772215"
 			(at 124.46 58.42 0)
 			(hide yes)
@@
 				)
 				(justify bottom)
+			)
+		)
+		(property "Part_Number" "SSK02-FPH-254-A2"
+			(at 124.46 58.42 0)
+			(hide yes)
+			(show_name no)
+			(do_not_autoplace no)
+			(effects
+				(font
+					(size 1.27 1.27)
+				)
 			)
 		)
@@
 			)
 		)
-		(property "Datasheet" ""
+		(property "Datasheet" "https://www.digikey.com/en/products/detail/same-sky-formerly-cui-devices/SSK02-FPH-254-A3/28772125"
 			(at 78.74 78.74 0)
 			(hide yes)
@@
 				)
 				(justify bottom)
+			)
+		)
+		(property "Part_Number" "SSK02-FPH-254-A3"
+			(at 78.74 78.74 90)
+			(hide yes)
+			(show_name no)
+			(do_not_autoplace no)
+			(effects
+				(font
+					(size 1.27 1.27)
+				)
 			)
 		)
@@
 			)
 		)
-		(property "Datasheet" ""
+		(property "Datasheet" "https://www.digikey.com/en/products/detail/same-sky-formerly-cui-devices/SSK02-FPH-254-A3/28772125"
 			(at 78.74 113.03 0)
 			(hide yes)
@@
 				)
 				(justify bottom)
+			)
+		)
+		(property "Part_Number" "SSK02-FPH-254-A3"
+			(at 78.74 113.03 90)
+			(hide yes)
+			(show_name no)
+			(do_not_autoplace no)
+			(effects
+				(font
+					(size 1.27 1.27)
+				)
 			)
 		)
@@
 			)
 		)
+		(property "Part_Number" ""
+			(at 170.18 127 0)
+			(hide yes)
+			(show_name no)
+			(do_not_autoplace no)
+			(effects
+				(font
+					(size 1.27 1.27)
+				)
+			)
+		)
 		(pin "1"
 		)
@@
 			)
 		)
-		(property "Datasheet" ""
+		(property "Datasheet" "https://www.digikey.com/en/products/detail/same-sky-formerly-cui-devices/SSK02-FPH-254-A3/28772125"
 			(at 78.74 39.37 0)
 			(hide yes)
@@
 				)
 				(justify bottom)
+			)
+		)
+		(property "Part_Number" "SSK02-FPH-254-A3"
+			(at 78.74 39.37 90)
+			(hide yes)
+			(show_name no)
+			(do_not_autoplace no)
+			(effects
+				(font
+					(size 1.27 1.27)
+				)
 			)
 		)
@@
 			)
 		)
+		(property "Part_Number" ""
+			(at 99.06 59.69 0)
+			(hide yes)
+			(show_name no)
+			(do_not_autoplace no)
+			(effects
+				(font
+					(size 1.27 1.27)
+				)
+			)
+		)
 		(pin "S1"
 		)
@@
 			)
 		)
-		(property "Datasheet" ""
+		(property "Datasheet" "https://www.digikey.com/en/products/detail/same-sky-formerly-cui-devices/SSK02-FPH-254-A3/28772125"
 			(at 78.74 144.78 0)
 			(hide yes)
@@
 				)
 				(justify bottom)
+			)
+		)
+		(property "Part_Number" "SSK02-FPH-254-A3"
+			(at 78.74 144.78 90)
+			(hide yes)
+			(show_name no)
+			(do_not_autoplace no)
+			(effects
+				(font
+					(size 1.27 1.27)
+				)
 			)
 		)
@@
 			)
 		)
+		(property "Part_Number" ""
+			(at 99.06 130.81 0)
+			(hide yes)
+			(show_name no)
+			(do_not_autoplace no)
+			(effects
+				(font
+					(size 1.27 1.27)
+				)
+			)
+		)
 		(pin "S1"
 		)
@@
 			(at 170.18 83.82 0)
 			(hide yes)
+			(show_name no)
+			(do_not_autoplace no)
+			(effects
+				(font
+					(size 1.27 1.27)
+				)
+			)
+		)
+		(property "Part_Number" ""
+			(at 170.18 83.82 0)
+			(hide yes)
