File: KiCad/PowerSystem.kicad_sch (KiCad schematic)
At the start: 6 parts, among them U1 LT1054

Commit message: Updates for 10_18_26
Other:
- moved on the sheet: BT1, C26
Changed lines of the file:
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@@
 	)
 	(junction
-		(at 101.6 72.39)
-		(diameter 0)
-		(color 0 0 0 0)
-	)
-	(junction
-		(at 101.6 92.71)
+		(at 91.44 72.39)
 		(diameter 0)
 		(color 0 0 0 0)
@@
 	)
 	(junction
+		(at 100.33 72.39)
+		(diameter 0)
+		(color 0 0 0 0)
+	)
+	(junction
 		(at 109.22 72.39)
 		(diameter 0)
@@
 	)
 	(junction
-		(at 93.98 72.39)
+		(at 100.33 92.71)
 		(diameter 0)
 		(color 0 0 0 0)
@@
 	(wire
 		(pts
-			(xy 101.6 76.2) (xy 101.6 72.39)
-		)
-		(stroke
-			(width 0)
-			(type default)
-		)
-	)
-	(wire
-		(pts
-			(xy 82.55 72.39) (xy 93.98 72.39)
+			(xy 100.33 78.74) (xy 100.33 72.39)
+		)
+		(stroke
+			(width 0)
+			(type default)
+		)
+	)
+	(wire
+		(pts
+			(xy 82.55 72.39) (xy 91.44 72.39)
 		)
 		(stroke
@@
 	(wire
 		(pts
-			(xy 93.98 76.2) (xy 93.98 72.39)
+			(xy 100.33 72.39) (xy 109.22 72.39)
+		)
+		(stroke
+			(width 0)
+			(type default)
+		)
+	)
+	(wire
+		(pts
+			(xy 91.44 76.2) (xy 91.44 72.39)
 		)
 		(stroke
@@
 	(wire
 		(pts
-			(xy 101.6 72.39) (xy 109.22 72.39)
-		)
-		(stroke
-			(width 0)
-			(type default)
-		)
-	)
-	(wire
-		(pts
 			(xy 124.46 93.98) (xy 124.46 92.71)
 		)
@@
 	(wire
 		(pts
-			(xy 101.6 92.71) (xy 109.22 92.71)
-		)
-		(stroke
-			(width 0)
-			(type default)
-		)
-	)
-	(wire
-		(pts
-			(xy 93.98 83.82) (xy 93.98 92.71)
-		)
-		(stroke
-			(width 0)
-			(type default)
-		)
-	)
-	(wire
-		(pts
-			(xy 101.6 81.28) (xy 101.6 92.71)
-		)
-		(stroke
-			(width 0)
-			(type default)
-		)
-	)
-	(wire
-		(pts
-			(xy 93.98 72.39) (xy 101.6 72.39)
+			(xy 100.33 92.71) (xy 91.44 92.71)
+		)
+		(stroke
+			(width 0)
+			(type default)
+		)
+	)
+	(wire
+		(pts
+			(xy 91.44 72.39) (xy 100.33 72.39)
+		)
+		(stroke
+			(width 0)
+			(type default)
+		)
+	)
+	(wire
+		(pts
+			(xy 91.44 83.82) (xy 91.44 92.71)
+		)
+		(stroke
+			(width 0)
+			(type default)
+		)
+	)
+	(wire
+		(pts
+			(xy 100.33 83.82) (xy 100.33 92.71)
 		)
 		(stroke
@@
 	(wire
 		(pts
-			(xy 101.6 92.71) (xy 93.98 92.71)
+			(xy 100.33 92.71) (xy 109.22 92.71)
 		)
 		(stroke
@@
 	(symbol
 		(lib_id "Device:C_Polarized_Small_US")
-		(at 101.6 78.74 0)
+		(at 100.33 81.28 0)
 		(unit 1)
 		(body_style 1)
@@
 		(dnp no)
 		(property "Reference" "C26"
-			(at 97.282 80.518 0)
+			(at 96.012 76.708 0)
 			(show_name no)
 			(do_not_autoplace no)
@@
 		)
 		(property "Value" "1uF"
-			(at 97.536 82.296 0)
+			(at 96.012 78.486 0)
 			(show_name no)
 			(do_not_autoplace no)
@@
 		)
 		(property "Footprint" "Capacitor_SMD:CP_Elec_4x5.7"
-			(at 101.6 78.74 0)
+			(at 100.33 81.28 0)
 			(hide yes)
 			(show_name no)
@@
 		)
 		(property "Datasheet" ""
-			(at 101.6 78.74 0)
+			(at 100.33 81.28 0)
 			(hide yes)
 			(show_name no)
@@
 		)
 		(property "Description" "Polarized capacitor, small US symbol"
-			(at 101.6 78.74 0)
+			(at 100.33 81.28 0)
 			(hide yes)
 			(show_name no)
@@
 	(symbol
 		(lib_id "Device:Battery_Cell")
-		(at 93.98 81.28 0)
+		(at 91.44 81.28 0)
 		(unit 1)
 		(body_style 1)
@@
 		(dnp no)
 		(property "Reference" "BT1"
-			(at 87.376 78.74 0)
+			(at 84.836 78.74 0)
 			(show_name no)
 			(do_not_autoplace no)
@@
 		)
 		(property "Value" "9V"
-			(at 87.63 81.026 0)
+			(at 85.09 81.026 0)
 			(show_name no)
 			(do_not_autoplace no)
@@
 		)
 		(property "Footprint" "Battery:BatteryHolder_MPD_BA9VPC_1xPP3"
-			(at 93.98 79.756 90)
+			(at 91.44 79.756 90)
 			(hide yes)
 			(show_name no)
@@
 		)
 		(property "Datasheet" ""
-			(at 93.98 79.756 90)
+			(at 91.44 79.756 90)
 			(hide yes)
 			(show_name no)
@@
 		)
 		(property "Description" "Single-cell battery"
-			(at 93.98 81.28 0)
+			(at 91.44 81.28 0)
 			(hide yes)
 			(show_name no)
@@
 		)
 		(property "Sim.Device" "V"
-			(at 93.98 81.28 0)
+			(at 91.44 81.28 0)
 			(hide yes)
 			(show_name no)
@@
 		)
 		(property "Sim.Type" "DC"
-			(at 93.98 81.28 0)
+			(at 91.44 81.28 0)
 			(hide yes)
 			(show_name no)
@@
 		)
 		(property "Sim.Pins" "1=+ 2=-"
-			(at 93.98 81.28 0)
-			(hide yes)
-			(show_name no)
+			(at 91.44 81.28 0)
+			(hide yes)
+			(show_name no)

Commit message: Pushing PCB, and controls schem
Parts:
- added C28, C29, C30, C31, C32, C33, C34, C35: 1uF, Capacitor_SMD:C_0603_1608Metric, symbol Device:C
- added U12, U15: MCP1703T-3302E/DB, lin_reg:SOT-223_3MC_MCH, symbol MCP1703_3302:MCP1703T-3302E_DB
- added U13, U14: MCP1703T-5002E/DB, lin_reg_50:SOT-223_3MC_MCH, symbol MPC1703_500:MCP1703T-5002E_DB
Connections:
- net +9V: now also C28.1, C30.1, C32.1, C33.1, U12.1 (VIN), U13.1 (VIN), U14.1 (VIN), U15.1 (VIN)
- net GND: now also C28.2, C29.2, C30.2, C31.2, C32.2, C33.2, C34.2, C35.2, U12.2 (GND), U13.2 (GND), U14.2 (GND), U15.2 (GND)
- new net +3.3V: C35.1, U12.3 (VOUT)
- new net +3.3VA: C34.1, U15.3 (VOUT)
- new net +5VA: C31.1, U14.3 (VOUT)
- new net +5VD: C29.1, U13.3 (VOUT)
- no-connect marks 0 -> 3
Other:
- moved on the sheet: BT1, C24, C25, C26, C27, U1

Commit message: Best one yet
Parts:
- removed BT1: 9V, Battery:BatteryHolder_MPD_BA9VPC_1xPP3, symbol Device:Battery_Cell
- added J10: Battery in, SSK02-FPH-254-A2:SAMESKY_SSK02-FPH-254-A2, symbol female_headers_2pin:SSK02-FPH-254-A2
- added J11: P_Switch, SSK02-FPH-254-A2:SAMESKY_SSK02-FPH-254-A2, symbol female_headers_2pin:SSK02-FPH-254-A2
Connections:
- net +9V: now also J10.2, J11.1
- net GND: now also J11.2
- no-connect marks 3 -> 4

Commit message: A bunch of schematic changes
Parts:
- removed C32, C35: 1uF, Capacitor_SMD:C_0603_1608Metric, symbol Device:C
- removed J10: Battery in, SSK02-FPH-254-A2:SAMESKY_SSK02-FPH-254-A2, symbol female_headers_2pin:SSK02-FPH-254-A2
- removed J11: P_Switch, SSK02-FPH-254-A2:SAMESKY_SSK02-FPH-254-A2, symbol female_headers_2pin:SSK02-FPH-254-A2
- removed U12: MCP1703T-3302E/DB, lin_reg:SOT-223_3MC_MCH, symbol MCP1703_3302:MCP1703T-3302E_DB
- added BT2: Battery, symbol Device:Battery
- added J14: powerRailAndBatteryGround, SSK02-FPH-254-A2:SAMESKY_SSK02-FPH-254-A2, symbol female_headers_2pin:SSK02-FPH-254-A2
- added J15: Barrel_Jack_Switch, symbol Connector:Barrel_Jack_Switch
- added J16: Barrel3andbarrel2, SSK02-FPH-254-A2:SAMESKY_SSK02-FPH-254-A2, symbol female_headers_2pin:SSK02-FPH-254-A2
- added J18: positivePowerInputs, SSK02-FPH-254-A3:SAMESKY_SSK02-FPH-254-A3, symbol female_headers_3pin:SSK02-FPH-254-A3
- added SW8: SW_DIP_x01, symbol Switch:SW_DIP_x01
- added U2: PMEG2005CT_215, SOT_05CT215_NEX, symbol PowerDiode:PMEG2005CT_215
Connections:
- net +9V: now also J14.1, SW8.2
- net GND: now also J15.2, J16.2
- new net: J15.1, J18.3, U2.1 (anode)
- new net: BT2.2 (-), J14.2, J15.3, J16.1
- new net: BT2.1 (+), J18.2, U2.2 (anode)
- new net: J18.1, SW8.1, U2.3 (common_cathode)
- no-connect marks 4 -> 3

Commit message: First iteration, need to tweak some things
Parts:
- removed U13, U14: MCP1703T-5002E/DB, lin_reg_50:SOT-223_3MC_MCH, symbol MPC1703_500:MCP1703T-5002E_DB
- removed U15: MCP1703T-3302E/DB, lin_reg:SOT-223_3MC_MCH, symbol MCP1703_3302:MCP1703T-3302E_DB
- added U13, U14: MCP1703T-5002E/DB, lin_reg50:SOT-223_3MC_MCH, symbol lin_reg_5002:MCP1703T-5002E_DB
- added U15: MCP1703T-3302E/DB, lin_reg33:SOT-223_3MC_MCH, symbol lin_reg_330:MCP1703T-3302E_DB
- J14, J16: footprint SSK02-FPH-254-A2:SAMESKY_SSK02-FPH-254-A2 -> header_fem_pin2:SAMESKY_SSK02-FPH-254-A2
- J18: footprint SSK02-FPH-254-A3:SAMESKY_SSK02-FPH-254-A3 -> header_fem_pin3:SAMESKY_SSK02-FPH-254-A3
- U1: now in the parts list
- U2: footprint SOT_05CT215_NEX -> powa_protec_dat_diode:SOT_05CT215_NEX-M
Connections:
- net +3.3VA: now also U15.3 (VOUT)
- net +5VA: now also U14.3 (VOUT)
- net +5VD: now also U13.3 (VOUT)
- net +9V: now also U13.1 (VIN), U14.1 (VIN), U15.1 (VIN)
- net GND: now also U13.2 (GND), U14.2 (GND), U15.2 (GND)
Other:
- moved on the sheet: U2

Commit message: Changes to the BoM
Parts:
- C24: Part_Number (none) -> UWT1H100MCL1GB
- C25: Part_Number (none) -> 865080545012
- C26, C27: Part_Number (none) -> 865060640001
- C28, C29, C30, C31, C33, C34: Part_Number (none) -> C0603C105K4RACTU
- J14, J16: Part_Number (none) -> SSK02-FPH-254-A2
- J18: Part_Number (none) -> SSK02-FPH-254-A3
- U1: Part_Number (none) -> LT1054CDWR
- U13, U14: Part_Number (none) -> MCP1703-5002E/DB
- U15: Part_Number (none) -> MCP1703-3302E/DB
- U2: Part_Number (none) -> PMEG2005CT,215

Commit message: done
Parts:
- removed U1: LT1054, charge_pump:SOIC127P1030X265-16N, symbol Regulator_SwitchedCapacitor:LT1054
- added U1: LT1054CDWR, lt1054_16soic:DW16-M, symbol lt1054_soic16:LT1054CDWR
Connections:
- net +9V: now also U1.14 (VCC)
- net -9V: now also U1.11 (VOUT)
- net GND: now also U1.5 (GND)
- net at C24.1: now also U1.4 (CAP+)
- net at C24.2: now also U1.6 (CAP-)
- no-connect marks 3 -> 11
Other:
- moved on the sheet: C24, C25, C26, C27
